File: hw/rev1/FlightComputer/FlightComputer.kicad_pcb (KiCad board)
At the start: 2 copper layers, 103.7 x 148 mm, 421 parts, among them J1 SJ-43617-SMT, J10 Conn_DEBUG, J11 Conn_02x10_Odd_Even, J12 USB_B_Micro, J13 USB_B_Micro, J2 Conn_01x02, J3 Conn_01x02, J4 Conn_01x01, J5 ED060SC7_EPD, J6 RPI_Connector, J7 Micro_SD_Card, J8 Conn_01x02, J9 IPEX_IPX, M1 TEA5767_Radio_Module, M2 GY-91, M3 GY-86, SW1 SW_Push, SW10 SW_Push, SW11 SW_Push, SW2 SW_Push, SW3 SW_Push, SW4 SW_Push, SW5 SW_Push, SW6 SW_Push, SW7 SW_Push, SW8 SW_Push, SW9 SW_Push, U1 WM8960, U10 TPS61090, U11 TPS22917DBV, U12 Teseo-LIV3F, U13 STM32H745IIT, U14 STMPS2151STR, U15 USBLC6-2SC6, U16 USBLC6-2SC6, U2 TPS65186, U3 MT25QL512ABB8ESF, U4 MT48LC16M16A2P, U5 MAX809TTRG, U6 XC6220B331MR-G, U7 MCP73871, U8 XC6220B331MR-G, U9 XC6220B331MR-G, X1 24MHz, Y1 25MHz

Commit message: ...
Parts:
- removed C1, C100, C102, C103, C104, C105, C106, C107, C108, C109, C111, C112, C113, C114, C115, C116, C117, C118, C119, C16, C19, C2, C3, C41, C42, C43, C44, C45, C46, C47, C48, C49, C50, C51, C57, C63, C68, C70, C73, C74, C75, C76, C77, C78, C79, C80, C81, C82, C85, C86, C87, C88, C89, C94, C98: 0.1uF, Capacitor_SMD:C_0402_1005Metric
- removed C10, C11, C12, C13, C6, C7, C95: 220pF, Capacitor_SMD:C_0402_1005Metric
- removed C101, C120, C121, C17, C18, C20, C21, C22, C35, C96: 10uF, Capacitor_SMD:C_0603_1608Metric_Pad1.05x0.95mm_HandSolder
- removed C110, C14, C15, C4, C5, C91, C92, C93: 4.7uF, Capacitor_SMD:C_0603_1608Metric_Pad1.05x0.95mm_HandSolder
- removed C23, C24, C31, C32, C33, C34, C36, C37, C38, C39: 4.7uF, Capacitor_SMD:C_0402_1005Metric
- removed C25, C26: 0.1uF, Capacitor_SMD:C_0603_1608Metric_Pad1.05x0.95mm_HandSolder
- removed C27, C28: 0.01uF, Capacitor_SMD:C_0603_1608Metric_Pad1.05x0.95mm_HandSolder
- removed C29, C30, C61: 2.2uF, Capacitor_SMD:C_0402_1005Metric
- removed C40, C53, C54, C59, C65, C69, C90, C97, C99: 1uF, Capacitor_SMD:C_0402_1005Metric
- removed C52, C56, C58, C64, C67, C71, C8, C9: 10uF, Capacitor_Tantalum_SMD:CP_EIA-1608-08_AVX-J_Pad1.25x1.05mm_HandSolder
- removed C55, C60, C66: N/C, Capacitor_SMD:C_0402_1005Metric
- removed C62: 100uF, Capacitor_Tantalum_SMD:CP_EIA-3216-10_Kemet-I_Pad1.58x1.35mm_HandSolder
- removed C72: 22pF, Capacitor_SMD:C_0402_1005Metric
- removed C83, C84: 18pF, Capacitor_SMD:C_0402_1005Metric
- removed D1, D2: BAS3010S, FlightComputer_Library:TSLP-2-17
- removed D3, D4, D5, D6: BAT54-SOT23, Diode_SMD:D_SOT-23_ANK
- removed D7: LED_R, LED_SMD:LED_0603_1608Metric_Pad1.05x0.95mm_HandSolder
- removed D8, D9: LED_G, LED_SMD:LED_0603_1608Metric_Pad1.05x0.95mm_HandSolder
- removed FB1: BEAD(BMJ1608HM180NTR), Inductor_SMD:L_0603_1608Metric_Pad1.05x0.95mm_HandSolder
- removed J1: SJ-43617-SMT, FlightComputer_Library:SJ-43617-SMT
- removed J10: Conn_DEBUG, Connector_Molex:Molex_SPOX_5268-04A_1x04_P2.50mm_Horizontal
- removed J11: Conn_02x10_Odd_Even, Connector_PinHeader_2.54mm:PinHeader_2x10_P2.54mm_Vertical
- removed J12, J13: USB_B_Micro, Connector_USB:USB_Micro-B_Molex-105017-0001
- removed J2, J3, J8: Conn_01x02, Connector_Molex:Molex_SPOX_5268-02A_1x02_P2.50mm_Horizontal
- removed J4: Conn_01x01, Connector_Pin:Pin_D1.2mm_L10.2mm_W2.9mm_FlatFork
- removed J5: ED060SC7_EPD, FlightComputer_Library:AXT334124
- removed J6: RPI_Connector, Connector_PinSocket_2.54mm:PinSocket_2x20_P2.54mm_Vertical_SMD
- removed J7: Micro_SD_Card, Connector_Card:microSD_HC_Hirose_DM3AT-SF-PEJM5
- removed J9: IPEX_IPX, FlightComputer_Library:IPEX-IPX
- removed L1, L2, L3, L4, L5, L6, L7: Ferrite, Inductor_SMD:L_0402_1005Metric
- removed L10: 68uH w/2A, FlightComputer_Library:L_10x11mm
- removed L11: 33nH, Inductor_SMD:L_0402_1005Metric
- removed L12: 2.2uH (LQM2MPN2R2NG0), FlightComputer_Library:L_0806_2016Metric
- removed L8: 2.2uH, Inductor_SMD:L_Taiyo-Yuden_MD-4040
- removed L9: 4.7uH, FlightComputer_Library:L_1515(4040 metric)
- removed M1: TEA5767_Radio_Module, FlightComputer_Library:TEA5756-TJ-102BC
- removed M2: GY-91, FlightComputer_Library:GY-91
- removed M3: GY-86, FlightComputer_Library:GY-86
- removed R1, R113, R116, R120, R123, R127, R133, R136, R161, R162, R163, R164, R169, R170, R171, R172, R174, R175, R176, R183, R186, R188: 100K, Resistor_SMD:R_0402_1005Metric
- removed R10, R100, R101, R102, R107, R108, R109, R110, R111, R112, R122, R124, R126, R13, R131, R135, R141, R142, R143, R144, R145, R146, R147, R15, R150, R151, R152, R153, R154, R155, R156, R16, R17, R177, R178, R179, R180, R181, R182, R2, R206, R209, R210, R211, R212, R213, R214, R215, R216, R23, R24, R25, R26, R27, R28, R29, R3, R32, R33, R34, R35, R38, R39, R4, R40, R41, R42, R43, R44, R45, R47, R48, R49, R5, R50, R51, R52, R53, R54, R55, R56, R57, R58, R59, R6, R60, R61, R62, R63, R64, R65, R66, R67, R68, R69, R7, R70, R71, R72, R73, R74, R75, R76, R77, R78, R79, R8, R80, R81, R82, R83, R84, R85, R86, R87, R88, R89, R9, R90, R91, R92, R93, R94, R97, R98, R99: 33R, Resistor_SMD:R_0402_1005Metric
- removed R103, R104, R105, R106, R95, R96: 47K, Resistor_SMD:R_0402_1005Metric
- removed R11, R117, R12, R148, R149, R185, R193, R195, R198, R199, R200: N/C, Resistor_SMD:R_0402_1005Metric
- removed R114: 270K, Resistor_SMD:R_0402_1005Metric
- removed R115, R128, R140, R18, R20: 1M, Resistor_SMD:R_0402_1005Metric
- removed R118, R119, R134, R138, R157, R158, R159, R160, R165, R166, R167, R168, R173, R187, R217: 1K, Resistor_SMD:R_0402_1005Metric
- removed R121: 15K, Resistor_SMD:R_0402_1005Metric
- removed R125, R129: 1.87M, Resistor_SMD:R_0402_1005Metric
- removed R130, R132: 340K, Resistor_SMD:R_0402_1005Metric
- removed R137: 560K, Resistor_SMD:R_0402_1005Metric
- removed R139, R194, R196, R197, R201, R202, R203, R204, R205: 0R, Resistor_SMD:R_0402_1005Metric
- removed R14, R184, R189, R190, R191, R192, R207, R30, R31, R36, R37, R46: 10K, Resistor_SMD:R_0402_1005Metric
- removed R19: 47.5K, Resistor_SMD:R_0402_1005Metric
- removed R208: 47k, Resistor_SMD:R_0402_1005Metric
- removed R21: 52.3K, Resistor_SMD:R_0402_1005Metric
- removed R22: 43K, Resistor_SMD:R_0402_1005Metric
- removed SW1, SW2, SW3, SW4, SW5, SW6, SW7, SW8, SW9: SW_Push, Button_Switch_SMD:SW_SPST_B3S-1000
- removed SW10, SW11: SW_Push, Button_Switch_SMD:SW_Push_SPST_NO_Alps_SKRK
- removed TH1: NCP18XH103F03RB(10K), Resistor_SMD:R_0603_1608Metric_Pad1.05x0.95mm_HandSolder
- removed TP1: OUT3, TestPoint:TestPoint_Pad_D1.0mm
- removed TP10: GPS_WAKEUP, TestPoint:TestPoint_Pad_D1.0mm
- removed TP11: 1PPS, TestPoint:TestPoint_Pad_D1.0mm
- removed TP12: PA1, TestPoint:TestPoint_Pad_D1.0mm
- removed TP13: PC2, TestPoint:TestPoint_Pad_D1.0mm
- removed TP14: PC14, TestPoint:TestPoint_Pad_D1.0mm
- removed TP15: PC15, TestPoint:TestPoint_Pad_D1.0mm
- removed TP2: RINPUT3, TestPoint:TestPoint_Pad_D1.0mm
- removed TP3: EINK_SPI_SCL, TestPoint:TestPoint_Pad_D1.0mm
- removed TP4: EINK_SPI_SDI, TestPoint:TestPoint_Pad_D1.0mm
- removed TP5: EINK_SPI_CS, TestPoint:TestPoint_Pad_D1.0mm
- removed TP6: EINK_SPI_SDO, TestPoint:TestPoint_Pad_D1.0mm
- removed TP7: GPS_SCL, TestPoint:TestPoint_Pad_D1.0mm
- removed TP8: GPS_nRST, TestPoint:TestPoint_Pad_D1.0mm
- removed TP9: GPS_SDA, TestPoint:TestPoint_Pad_D1.0mm
- removed U1: WM8960, Package_DFN_QFN:QFN-32-1EP_5x5mm_P0.5mm_EP3.3x3.3mm_ThermalVias
- removed U10: TPS61090, Package_DFN_QFN:QFN-16-1EP_4x4mm_P0.65mm_EP2.5x2.5mm
- removed U11: TPS22917DBV, Package_TO_SOT_SMD:SOT-23-6
- removed U12: Teseo-LIV3F, FlightComputer_Library:Teseo-LIV3F
- removed U13: STM32H745IIT, Package_QFP:LQFP-176_24x24mm_P0.5mm
- removed U14: STMPS2151STR, Package_TO_SOT_SMD:SOT-23-5_HandSoldering
- removed U15, U16: USBLC6-2SC6, Package_TO_SOT_SMD:SOT-23-6_Handsoldering
- removed U2: TPS65186, Package_DFN_QFN:VQFN-48-1EP_7x7mm_P0.5mm_EP5.15x5.15mm_ThermalVias
- removed U3: MT25QL512ABB8ESF, FlightComputer_Library:SOP2-16_7.5x10.3mm_P1.27mm
- removed U4: MT48LC16M16A2P, Package_SO:TSOP-II-54_22.2x10.16mm_P0.8mm
- removed U5: MAX809TTRG, Package_TO_SOT_SMD:SOT-23
- removed U6, U8, U9: XC6220B331MR-G, Package_TO_SOT_SMD:SOT-23-5_HandSoldering
- removed U7: MCP73871, Package_DFN_QFN:QFN-20-1EP_4x4mm_P0.5mm_EP2.5x2.5mm
- removed X1: 24MHz, Oscillator:Oscillator_SMD_Abracon_ASE-4Pin_3.2x2.5mm_HandSoldering
- removed Y1: 25MHz, Crystal:Crystal_SMD_3225-4Pin_3.2x2.5mm_HandSoldering
Other:
- board size 103.7 x 148 mm -> 102 x 148 mm

Commit message: ...
Parts:
- added C1: 0.1uF, Capacitor_SMD:C_0402_1005Metric, F.Cu at (87.8, 70.1)
- added C10: 220pF, Capacitor_SMD:C_0402_1005Metric, F.Cu at (104.0, 95.5)
- added C100: 0.1uF, Capacitor_SMD:C_0402_1005Metric, F.Cu at (-37.6, 65.8)
- added C101: 10uF, Capacitor_SMD:C_0603_1608Metric_Pad1.05x0.95mm_HandSolder, F.Cu at (-47.1, 67.6)
- added C102: 0.1uF, Capacitor_SMD:C_0402_1005Metric, F.Cu at (-43.4, 74.3)
- added C103: 0.1uF, Capacitor_SMD:C_0402_1005Metric, F.Cu at (-43.4, 72.3)
- added C104: 0.1uF, Capacitor_SMD:C_0402_1005Metric, F.Cu at (-39.1, 68.3)
- added C105: 0.1uF, Capacitor_SMD:C_0402_1005Metric, F.Cu at (-36.2, 69.8)
- added C106: 0.1uF, Capacitor_SMD:C_0402_1005Metric, F.Cu at (-30.0, 61.8)
- added C107: 0.1uF, Capacitor_SMD:C_0402_1005Metric, F.Cu at (-40.5, 72.3)
- added C108: 0.1uF, Capacitor_SMD:C_0402_1005Metric, F.Cu at (-39.1, 70.3)
- added C109: 0.1uF, Capacitor_SMD:C_0402_1005Metric, F.Cu at (-34.7, 65.8)
- added C11: 220pF, Capacitor_SMD:C_0402_1005Metric, F.Cu at (106.6, 95.5)
- added C110: 4.7uF, Capacitor_SMD:C_0603_1608Metric_Pad1.05x0.95mm_HandSolder, F.Cu at (-42.3, 62.1)
- added C111: 0.1uF, Capacitor_SMD:C_0402_1005Metric, F.Cu at (-31.8, 63.8)
- added C112: 0.1uF, Capacitor_SMD:C_0402_1005Metric, F.Cu at (-36.2, 67.8)
- added C113: 0.1uF, Capacitor_SMD:C_0402_1005Metric, F.Cu at (-40.5, 74.3)
- added C114: 0.1uF, Capacitor_SMD:C_0402_1005Metric, F.Cu at (-34.7, 63.8)
- added C115: 0.1uF, Capacitor_SMD:C_0402_1005Metric, F.Cu at (-33.3, 67.8)
- added C116: 0.1uF, Capacitor_SMD:C_0402_1005Metric, F.Cu at (-31.8, 65.8)
- added C117: 0.1uF, Capacitor_SMD:C_0402_1005Metric, F.Cu at (-37.6, 72.3)
- added C118: 0.1uF, Capacitor_SMD:C_0402_1005Metric, F.Cu at (-28.9, 63.8)
- added C119: 0.1uF, Capacitor_SMD:C_0402_1005Metric, F.Cu at (-37.6, 74.3)
- added C12: 220pF, Capacitor_SMD:C_0402_1005Metric, F.Cu at (109.7, 95.8)
- added C120: 10uF, Capacitor_SMD:C_0603_1608Metric_Pad1.05x0.95mm_HandSolder, F.Cu at (-41.3, 103.7)
- added C121: 10uF, Capacitor_SMD:C_0603_1608Metric_Pad1.05x0.95mm_HandSolder, F.Cu at (136.0, 33.7)
- added C13: 220pF, Capacitor_SMD:C_0402_1005Metric, F.Cu at (112.7, 95.4)
- added C14: 4.7uF, Capacitor_SMD:C_0603_1608Metric_Pad1.05x0.95mm_HandSolder, F.Cu at (87.9, 79.7)
- added C15: 4.7uF, Capacitor_SMD:C_0603_1608Metric_Pad1.05x0.95mm_HandSolder, F.Cu at (87.7, 81.9)
- added C16: 0.1uF, Capacitor_SMD:C_0402_1005Metric, F.Cu at (105.5, 86.4)
- added C17: 10uF, Capacitor_SMD:C_0603_1608Metric_Pad1.05x0.95mm_HandSolder, F.Cu at (149.5, 84.5)
- added C18: 10uF, Capacitor_SMD:C_0603_1608Metric_Pad1.05x0.95mm_HandSolder, F.Cu at (149.7, 87.5)
- added C19: 0.1uF, Capacitor_SMD:C_0402_1005Metric, F.Cu at (156.3, 85.4)
- added C2: 0.1uF, Capacitor_SMD:C_0402_1005Metric, F.Cu at (87.9, 71.6)
- added C20: 10uF, Capacitor_SMD:C_0603_1608Metric_Pad1.05x0.95mm_HandSolder, F.Cu at (158.8, 87.3)
- added C21: 10uF, Capacitor_SMD:C_0603_1608Metric_Pad1.05x0.95mm_HandSolder, F.Cu at (-43.9, 53.1)
- added C22: 10uF, Capacitor_SMD:C_0603_1608Metric_Pad1.05x0.95mm_HandSolder, F.Cu at (-40.3, 47.6)
- added C23: 4.7uF, Capacitor_SMD:C_0402_1005Metric, F.Cu at (-28.8, 44.8)
- added C24: 4.7uF, Capacitor_SMD:C_0402_1005Metric, F.Cu at (-15.8, 40.8)
- added C25: 0.1uF, Capacitor_SMD:C_0603_1608Metric_Pad1.05x0.95mm_HandSolder, F.Cu at (-25.4, 37.1)
- added C26: 0.1uF, Capacitor_SMD:C_0603_1608Metric_Pad1.05x0.95mm_HandSolder, F.Cu at (-49.6, 56.5)
- added C27: 0.01uF, Capacitor_SMD:C_0603_1608Metric_Pad1.05x0.95mm_HandSolder, F.Cu at (-45.3, 56.5)
- added C28: 0.01uF, Capacitor_SMD:C_0603_1608Metric_Pad1.05x0.95mm_HandSolder, F.Cu at (-40.3, 50.1)
- added C29: 2.2uF, Capacitor_SMD:C_0402_1005Metric, F.Cu at (-18.8, 36.8)
- added C3: 0.1uF, Capacitor_SMD:C_0402_1005Metric, F.Cu at (88.0, 72.9)
- added C30: 2.2uF, Capacitor_SMD:C_0402_1005Metric, F.Cu at (-14.3, 44.8)
- added C31: 4.7uF, Capacitor_SMD:C_0402_1005Metric, F.Cu at (-22.0, 52.4)
- added C32: 4.7uF, Capacitor_SMD:C_0402_1005Metric, F.Cu at (-18.6, 47.9)
- added C33: 4.7uF, Capacitor_SMD:C_0402_1005Metric, F.Cu at (-24.9, 54.8)
- added C34: 4.7uF, Capacitor_SMD:C_0402_1005Metric, F.Cu at (-14.3, 42.8)
- added C35: 10uF, Capacitor_SMD:C_0603_1608Metric_Pad1.05x0.95mm_HandSolder, F.Cu at (-34.6, 44.2)
- added C36: 4.7uF, Capacitor_SMD:C_0402_1005Metric, F.Cu at (-21.5, 50.4)
- added C37: 4.7uF, Capacitor_SMD:C_0402_1005Metric, F.Cu at (-17.2, 45.9)
- added C38: 4.7uF, Capacitor_SMD:C_0402_1005Metric, F.Cu at (-24.9, 52.8)
- added C39: 4.7uF, Capacitor_SMD:C_0402_1005Metric, F.Cu at (-21.5, 48.4)
- added C4: 4.7uF, Capacitor_SMD:C_0603_1608Metric_Pad1.05x0.95mm_HandSolder, F.Cu at (87.9, 75.9)
- added C40: 1uF, Capacitor_SMD:C_0402_1005Metric, F.Cu at (6.71, 15.9)
- added C41: 0.1uF, Capacitor_SMD:C_0402_1005Metric, F.Cu at (6.60, 17.4)
- added C42: 0.1uF, Capacitor_SMD:C_0402_1005Metric, F.Cu at (88.6, 52.8)
- added C43: 0.1uF, Capacitor_SMD:C_0402_1005Metric, F.Cu at (36.7, 69.2)
- added C44: 0.1uF, Capacitor_SMD:C_0402_1005Metric, F.Cu at (38.2, 69.3)
- added C45: 0.1uF, Capacitor_SMD:C_0402_1005Metric, F.Cu at (39.5, 69.2)
- added C46: 0.1uF, Capacitor_SMD:C_0402_1005Metric, F.Cu at (41.3, 69.3)
- added C47: 0.1uF, Capacitor_SMD:C_0402_1005Metric, F.Cu at (42.7, 69.3)
- added C48: 0.1uF, Capacitor_SMD:C_0402_1005Metric, F.Cu at (44.1, 69.4)
- added C49: 0.1uF, Capacitor_SMD:C_0402_1005Metric, F.Cu at (45.5, 69.5)
- added C5: 4.7uF, Capacitor_SMD:C_0603_1608Metric_Pad1.05x0.95mm_HandSolder, F.Cu at (87.9, 77.7)
- added C50: 0.1uF, Capacitor_SMD:C_0402_1005Metric, F.Cu at (99.3, 122.2)
- added C51: 0.1uF, Capacitor_SMD:C_0402_1005Metric, F.Cu at (83.8, 16.3)
- added C52: 10uF, Capacitor_Tantalum_SMD:CP_EIA-1608-08_AVX-J_Pad1.25x1.05mm_HandSolder, F.Cu at (83.4, 13.5)
- added C53: 1uF, Capacitor_SMD:C_0402_1005Metric, F.Cu at (75.3, 18.5)
- added C54: 1uF, Capacitor_SMD:C_0402_1005Metric, F.Cu at (78.4, 18.3)
- added C55: N/C, Capacitor_SMD:C_0402_1005Metric, F.Cu at (83.2, 18.3)
- added C56: 10uF, Capacitor_Tantalum_SMD:CP_EIA-1608-08_AVX-J_Pad1.25x1.05mm_HandSolder, F.Cu at (-78.0, 41.6)
- added C57: 0.1uF, Capacitor_SMD:C_0402_1005Metric, F.Cu at (-78.0, 57.3)
- added C58: 10uF, Capacitor_Tantalum_SMD:CP_EIA-1608-08_AVX-J_Pad1.25x1.05mm_HandSolder, F.Cu at (-86.0, 49.8)
- added C59: 1uF, Capacitor_SMD:C_0402_1005Metric, F.Cu at (-79.4, 47.4)
- added C6: 220pF, Capacitor_SMD:C_0402_1005Metric, F.Cu at (93.4, 96.1)
- added C60: N/C, Capacitor_SMD:C_0402_1005Metric, F.Cu at (-70.6, 49.1)
- added C61: 2.2uF, Capacitor_SMD:C_0402_1005Metric, F.Cu at (-73.5, 51.9)
- added C62: 100uF, Capacitor_Tantalum_SMD:CP_EIA-3216-10_Kemet-I_Pad1.58x1.35mm_HandSolder, F.Cu at (120.5, 31.6)
- added C67: 10uF, Capacitor_Tantalum_SMD:CP_EIA-1608-08_AVX-J_Pad1.25x1.05mm_HandSolder, F.Cu at (-78.0, 38.9)
- added C68: 0.1uF, Capacitor_SMD:C_0402_1005Metric, F.Cu at (-67.8, 45.1)
- added C69: 1uF, Capacitor_SMD:C_0402_1005Metric, F.Cu at (55.9, 14.7)
- added C7: 220pF, Capacitor_SMD:C_0402_1005Metric, F.Cu at (98.0, 95.6)
- added C70: 0.1uF, Capacitor_SMD:C_0402_1005Metric, F.Cu at (62.7, 16.0)
- added C71: 10uF, Capacitor_Tantalum_SMD:CP_EIA-1608-08_AVX-J_Pad1.25x1.05mm_HandSolder, F.Cu at (66.4, 15.5)
- added C72: N/C, Capacitor_SMD:C_0402_1005Metric, F.Cu at (59.2, 16.3)
- added C8: 10uF, Capacitor_Tantalum_SMD:CP_EIA-1608-08_AVX-J_Pad1.25x1.05mm_HandSolder, F.Cu at (93.4, 91.7)
- added C83: 18pF, Capacitor_SMD:C_0402_1005Metric, F.Cu at (44.0, 28.5)
- added C84: 18pF, Capacitor_SMD:C_0402_1005Metric, F.Cu at (44.2, 29.8)
- added C85: 0.1uF, Capacitor_SMD:C_0402_1005Metric, F.Cu at (10.0, 68.1)
- added C86: 0.1uF, Capacitor_SMD:C_0402_1005Metric, F.Cu at (8.20, 59.5)
- added C87: 0.1uF, Capacitor_SMD:C_0402_1005Metric, F.Cu at (-30.4, 67.8)
- added C88: 0.1uF, Capacitor_SMD:C_0402_1005Metric, F.Cu at (-28.9, 65.8)
- added C89: 0.1uF, Capacitor_SMD:C_0402_1005Metric, F.Cu at (-34.7, 71.8)
- added C9: 10uF, Capacitor_Tantalum_SMD:CP_EIA-1608-08_AVX-J_Pad1.25x1.05mm_HandSolder, F.Cu at (98.0, 91.7)
- added C90: 1uF, Capacitor_SMD:C_0402_1005Metric, F.Cu at (-44.9, 69.9)
- added C91: 4.7uF, Capacitor_SMD:C_0603_1608Metric_Pad1.05x0.95mm_HandSolder, F.Cu at (-46.7, 62.1)
- added C92: 4.7uF, Capacitor_SMD:C_0603_1608Metric_Pad1.05x0.95mm_HandSolder, F.Cu at (-51.4, 65.1)
- added C93: 4.7uF, Capacitor_SMD:C_0603_1608Metric_Pad1.05x0.95mm_HandSolder, F.Cu at (-51.4, 67.6)
- added C94: 0.1uF, Capacitor_SMD:C_0402_1005Metric, F.Cu at (-52.2, 72.4)
- added C95: 220pF, Capacitor_SMD:C_0402_1005Metric, F.Cu at (-38.7, 61.8)
- added C96: 10uF, Capacitor_SMD:C_0603_1608Metric_Pad1.05x0.95mm_HandSolder, F.Cu at (-47.1, 65.1)
- added C97: 1uF, Capacitor_SMD:C_0402_1005Metric, F.Cu at (-52.2, 74.4)
- added C98: 0.1uF, Capacitor_SMD:C_0402_1005Metric, F.Cu at (-43.5, 66.3)
- added C99: 1uF, Capacitor_SMD:C_0402_1005Metric, F.Cu at (-47.8, 69.9)
- added D1: MBR130T1G, Diode_SMD:D_SOD-123, F.Cu at (-48.9, 53.5)
- added D2: MBR130T1G, Diode_SMD:D_SOD-123, F.Cu at (-39.6, 44.6)
- added D3: RB531SM, Diode_SMD:D_SOD-523, F.Cu at (-32.0, 46.7)
- added D4: RB531SM, Diode_SMD:D_SOD-523, F.Cu at (-36.4, 50.1)
- added D5: RB531SM, Diode_SMD:D_SOD-523, F.Cu at (-30.6, 42.6)
- added D6: BAT54-SOT23, Diode_SMD:D_SOD-523, F.Cu at (-39.9, 52.6)
- added D7: LED_R, LED_SMD:LED_0603_1608Metric_Pad1.05x0.95mm_HandSolder, F.Cu at (-78.6, 45.1)
- added D8: LED_G, LED_SMD:LED_0603_1608Metric_Pad1.05x0.95mm_HandSolder, F.Cu at (-86.0, 52.4)
- added D9: LED_G, LED_SMD:LED_0603_1608Metric_Pad1.05x0.95mm_HandSolder, F.Cu at (-54.9, 24.9)
- added FB1: BEAD(BMJ1608HM180NTR), Inductor_SMD:L_0603_1608Metric_Pad1.05x0.95mm_HandSolder, F.Cu at (-51.4, 70.1)
- added J1: Conn_01x10, Connector_PinSocket_2.54mm:PinSocket_1x10_P2.54mm_Vertical, F.Cu at (91.3, 99.5)
- added J11: Conn_02x20_Odd_Even, Connector_PinSocket_2.54mm:PinSocket_2x20_P2.54mm_Vertical, F.Cu at (97.4, 5.21)
- added J12: USB_B_Micro, Connector_USB:USB_Micro-B_Molex-105017-0001, F.Cu at (144.6, 8.98)
- added J13: USB_B_Micro, Connector_USB:USB_Micro-B_Molex-105017-0001, F.Cu at (144.7, 27.4)
- added J2: Conn_01x10, Connector_PinSocket_2.54mm:PinSocket_1x10_P2.54mm_Vertical, F.Cu at (31.3, 99.5)
- added J4: Conn_01x01, Connector_Pin:Pin_D1.2mm_L10.2mm_W2.9mm_FlatFork, F.Cu at (128.7, 99.6)
- added J5: ED060SC7_EPD, FlightComputer_Library:AXT334124, F.Cu at (14.4, 16.2)
- added J6: RPI_Connector, Connector_PinSocket_2.54mm:PinSocket_2x20_P2.54mm_Vertical, F.Cu at (122.8, 41.4)
- added J7: Micro_SD_Card, Connector_Card:microSD_HC_Hirose_DM3AT-SF-PEJM5, F.Cu at (139.0, 61.0)
- added J8: Conn_01x02, Connector_Molex:Molex_SPOX_5268-02A_1x02_P2.50mm_Horizontal, F.Cu at (112.6, 8.65)
- added L1: Ferrite, Inductor_SMD:L_0402_1005Metric, F.Cu at (93.5, 94.1)
- added L10: 68uH w/2A, FlightComputer_Library:L_10x11mm, F.Cu at (107.5, 28.7)
- added L12: 2.2uH (LQM2MPN2R2NG0), FlightComputer_Library:L_0806_2016Metric, F.Cu at (-51.2, 62.3)
- added L2: Ferrite, Inductor_SMD:L_0402_1005Metric, F.Cu at (98.0, 93.8)
- added L3: Ferrite, Inductor_SMD:L_0402_1005Metric, F.Cu at (103.9, 93.8)
- added L4: Ferrite, Inductor_SMD:L_0402_1005Metric, F.Cu at (106.6, 93.8)
- added L5: Ferrite, Inductor_SMD:L_0402_1005Metric, F.Cu at (110.0, 93.9)
- added L6: Ferrite, Inductor_SMD:L_0402_1005Metric, F.Cu at (112.8, 93.7)
- added L7: Ferrite, Inductor_SMD:L_0402_1005Metric, F.Cu at (157.1, 83.4)
- added L8: 2.2uH, Inductor_SMD:L_Taiyo-Yuden_MD-4040, F.Cu at (6.90, 41.7)
- added L9: 4.7uH, FlightComputer_Library:L_1515(4040 metric), F.Cu at (17.1, 51.1)
- added M1: TEA5767_Radio_Module, FlightComputer_Library:TEA5756-TJ-102BC, F.Cu at (138.4, 85.4)
- added M2: GY-91, FlightComputer_Library:GY-91, F.Cu at (28.6, 84.6)
- added M3: GY-86, FlightComputer_Library:GY-86, F.Cu at (11.1, 84.8)
- added R10: 33R, Resistor_SMD:R_0402_1005Metric, F.Cu at (103.7, 69.6)
- added R100: 33R, Resistor_SMD:R_0402_1005Metric, F.Cu at (66.2, 114.3)
- added R101: 33R, Resistor_SMD:R_0402_1005Metric, F.Cu at (105.1, 116.2)
- added R102: 33R, Resistor_SMD:R_0402_1005Metric, F.Cu at (102.2, 118.2)
- added R103: 47K, Resistor_SMD:R_0402_1005Metric, F.Cu at (105.1, 114.2)
- added R104: 47K, Resistor_SMD:R_0402_1005Metric, F.Cu at (66.2, 116.3)
- added R105: 47K, Resistor_SMD:R_0402_1005Metric, F.Cu at (99.3, 116.2)
- added R106: 47K, Resistor_SMD:R_0402_1005Metric, F.Cu at (102.2, 114.2)
- added R107: 33R, Resistor_SMD:R_0402_1005Metric, F.Cu at (99.3, 114.2)
- added R108: 33R, Resistor_SMD:R_0402_1005Metric, F.Cu at (86.9, 115.4)
- added R109: 33R, Resistor_SMD:R_0402_1005Metric, F.Cu at (108.0, 114.2)
- added R11: N/C, Resistor_SMD:R_0402_1005Metric, F.Cu at (103.9, 71.0)
- added R110: 33R, Resistor_SMD:R_0402_1005Metric, F.Cu at (99.3, 124.2)
- added R111: 33R, Resistor_SMD:R_0402_1005Metric, F.Cu at (89.8, 117.4)
- added R112: 33R, Resistor_SMD:R_0402_1005Metric, F.Cu at (102.2, 120.2)
- added R113: 100K, Resistor_SMD:R_0402_1005Metric, F.Cu at (69.1, 114.3)
- added R114: 270K, Resistor_SMD:R_0402_1005Metric, F.Cu at (-73.5, 47.9)
- added R115: 1M, Resistor_SMD:R_0402_1005Metric, F.Cu at (75.2, 17.1)
- added R116: 100K, Resistor_SMD:R_0402_1005Metric, F.Cu at (-70.7, 45.1)
- added R117: N/C, Resistor_SMD:R_0402_1005Metric, F.Cu at (-76.4, 55.4)
- added R118: 1K, Resistor_SMD:R_0402_1005Metric, F.Cu at (-82.2, 54.5)
- added R119: 1K, Resistor_SMD:R_0402_1005Metric, F.Cu at (-76.4, 49.4)
- added R12: N/C, Resistor_SMD:R_0402_1005Metric, F.Cu at (103.8, 72.5)
- added R120: 100K, Resistor_SMD:R_0402_1005Metric, F.Cu at (-73.6, 45.9)
- added R121: 15K, Resistor_SMD:R_0402_1005Metric, F.Cu at (-69.2, 43.1)
- added R122: 33R, Resistor_SMD:R_0402_1005Metric, F.Cu at (-82.2, 56.5)
- added R123: 100K, Resistor_SMD:R_0402_1005Metric, F.Cu at (-79.3, 53.4)
- added R124: 33R, Resistor_SMD:R_0402_1005Metric, F.Cu at (-83.8, 58.7)
- added R125: 1.87M, Resistor_SMD:R_0402_1005Metric, F.Cu at (-79.3, 51.4)
- added R126: N/C, Resistor_SMD:R_0402_1005Metric, F.Cu at (-73.5, 53.9)
- added R128: 1M, Resistor_SMD:R_0402_1005Metric, F.Cu at (-86.7, 59.2)
- added R129: 1.87M, Resistor_SMD:R_0402_1005Metric, F.Cu at (-88.1, 57.2)
- added R13: 33R, Resistor_SMD:R_0402_1005Metric, F.Cu at (103.4, 74.5)
- added R130: 340K, Resistor_SMD:R_0402_1005Metric, F.Cu at (-71.4, 41.1)
- added R131: 33R, Resistor_SMD:R_0402_1005Metric, F.Cu at (-69.9, 38.6)
- added R132: 340K, Resistor_SMD:R_0402_1005Metric, F.Cu at (-82.4, 52.5)
- added R133: 100K, Resistor_SMD:R_0402_1005Metric, F.Cu at (-85.2, 54.7)
- added R134: 1K, Resistor_SMD:R_0402_1005Metric, F.Cu at (62.9, 14.5)
- added R135: 33R, Resistor_SMD:R_0402_1005Metric, F.Cu at (55.8, 16.5)
- added R136: 100K, Resistor_SMD:R_0402_1005Metric, F.Cu at (59.0, 14.7)
- added R137: 560K, Resistor_SMD:R_0402_1005Metric, F.Cu at (-43.6, 23.2)
- added R138: 1K, Resistor_SMD:R_0402_1005Metric, F.Cu at (-54.6, 26.8)
- added R139: 0R, Resistor_SMD:R_0402_1005Metric, F.Cu at (-46.0, 24.1)
- added R14: 10K, Resistor_SMD:R_0402_1005Metric, F.Cu at (105.2, 84.9)
- added R140: 1M, Resistor_SMD:R_0402_1005Metric, F.Cu at (-43.6, 24.9)
- added R141: 33R, Resistor_SMD:R_0402_1005Metric, F.Cu at (24.1, 98.9)
- added R142: 33R, Resistor_SMD:R_0402_1005Metric, F.Cu at (23.9, 100.2)
- added R143: 33R, Resistor_SMD:R_0402_1005Metric, F.Cu at (23.8, 101.4)
- added R144: 33R, Resistor_SMD:R_0402_1005Metric, F.Cu at (23.7, 102.8)
- added R145: 33R, Resistor_SMD:R_0402_1005Metric, F.Cu at (23.8, 104.7)
- added R146: 33R, Resistor_SMD:R_0402_1005Metric, F.Cu at (46.0, 95.8)
- added R147: 33R, Resistor_SMD:R_0402_1005Metric, F.Cu at (46.0, 94.6)
- added R148: N/C, Resistor_SMD:R_0402_1005Metric, F.Cu at (18.8, 99.7)
- added R149: N/C, Resistor_SMD:R_0402_1005Metric, F.Cu at (18.8, 101.3)
- added R15: 33R, Resistor_SMD:R_0402_1005Metric, F.Cu at (108.8, 84.8)
- added R150: 33R, Resistor_SMD:R_0402_1005Metric, F.Cu at (13.5, 98.7)
- added R151: 33R, Resistor_SMD:R_0402_1005Metric, F.Cu at (13.3, 101.1)
- added R152: 33R, Resistor_SMD:R_0402_1005Metric, F.Cu at (13.3, 103.2)
- added R153: 33R, Resistor_SMD:R_0402_1005Metric, F.Cu at (13.3, 104.7)
- added R154: 33R, Resistor_SMD:R_0402_1005Metric, F.Cu at (13.7, 105.8)
- added R155: 33R, Resistor_SMD:R_0402_1005Metric, F.Cu at (42.1, 94.7)
- added R156: 33R, Resistor_SMD:R_0402_1005Metric, F.Cu at (41.8, 96.5)
- added R157: 0R, Resistor_SMD:R_0402_1005Metric, F.Cu at (87.2, 8.60)
- added R158: 0R, Resistor_SMD:R_0402_1005Metric, F.Cu at (84.6, 8.70)
- added R159: 0R, Resistor_SMD:R_0402_1005Metric, F.Cu at (92.4, 8.62)
- added R16: 33R, Resistor_SMD:R_0402_1005Metric, F.Cu at (159.4, 83.4)
- added R160: 0R, Resistor_SMD:R_0402_1005Metric, F.Cu at (89.8, 8.60)
- added R165: 0R, Resistor_SMD:R_0402_1005Metric, F.Cu at (82.1, 8.60)
- added R166: 0R, Resistor_SMD:R_0402_1005Metric, F.Cu at (77.2, 8.40)
- added R167: 0R, Resistor_SMD:R_0402_1005Metric, F.Cu at (74.6, 8.40)
- added R168: 0R, Resistor_SMD:R_0402_1005Metric, F.Cu at (72.1, 8.20)
- added R17: 33R, Resistor_SMD:R_0402_1005Metric, F.Cu at (159.1, 85.4)
- added R173: 0R, Resistor_SMD:R_0402_1005Metric, F.Cu at (79.5, 8.60)
- added R177: 33R, Resistor_SMD:R_0402_1005Metric, F.Cu at (66.8, 8.30)
- added R178: 33R, Resistor_SMD:R_0402_1005Metric, F.Cu at (64.2, 8.30)
- added R179: 33R, Resistor_SMD:R_0402_1005Metric, F.Cu at (61.8, 8.40)
- added R18: 1M, Resistor_SMD:R_0402_1005Metric, F.Cu at (-21.6, 41.9)
- added R180: 33R, Resistor_SMD:R_0402_1005Metric, F.Cu at (59.3, 8.30)
- added R181: 33R, Resistor_SMD:R_0402_1005Metric, F.Cu at (56.8, 8.40)
- added R182: 33R, Resistor_SMD:R_0402_1005Metric, F.Cu at (54.2, 8.30)
- added R184: 10K, Resistor_SMD:R_0402_1005Metric, F.Cu at (42.6, 50.1)
- added R185: N/C, Resistor_SMD:R_0402_1005Metric, F.Cu at (42.9, 51.6)
- added R186: 100K, Resistor_SMD:R_0402_1005Metric, F.Cu at (10.0, 66.3)
- added R187: 1K, Resistor_SMD:R_0402_1005Metric, F.Cu at (10.7, 59.6)
- added R188: 100K, Resistor_SMD:R_0402_1005Metric, F.Cu at (8.52, 58.1)
- added R189: 10K, Resistor_SMD:R_0402_1005Metric, F.Cu at (-75.6, 78.6)
- added R19: 47.5K, Resistor_SMD:R_0402_1005Metric, F.Cu at (-33.7, 54.3)
- added R190: 10K, Resistor_SMD:R_0402_1005Metric, F.Cu at (-75.4, 75.8)
- added R191: 10K, Resistor_SMD:R_0402_1005Metric, F.Cu at (-75.6, 77.2)
- added R192: 10K, Resistor_SMD:R_0402_1005Metric, F.Cu at (-75.6, 79.8)
- added R193: N/C, Resistor_SMD:R_0402_1005Metric, F.Cu at (-33.3, 69.8)
- added R194: 0R, Resistor_SMD:R_0402_1005Metric, F.Cu at (-49.3, 72.4)
- added R195: N/C, Resistor_SMD:R_0402_1005Metric, F.Cu at (-40.6, 64.3)
- added R196: 0R, Resistor_SMD:R_0402_1005Metric, F.Cu at (-43.5, 64.3)
- added R197: 0R, Resistor_SMD:R_0402_1005Metric, F.Cu at (-35.8, 61.8)
- added R198: N/C, Resistor_SMD:R_0402_1005Metric, F.Cu at (-40.6, 66.3)
- added R199: N/C, Resistor_SMD:R_0402_1005Metric, F.Cu at (-49.3, 74.4)
- added R2: 33R, Resistor_SMD:R_0402_1005Metric, F.Cu at (108.0, 67.4)
- added R20: 1M, Resistor_SMD:R_0402_1005Metric, F.Cu at (-30.3, 50.9)
- added R200: N/C, Resistor_SMD:R_0402_1005Metric, F.Cu at (-46.3, 71.9)
- added R201: 0R, Resistor_SMD:R_0402_1005Metric, F.Cu at (-37.6, 63.8)
- added R202: 0R, Resistor_SMD:R_0402_1005Metric, F.Cu at (-42.0, 68.3)
- added R203: 0R, Resistor_SMD:R_0402_1005Metric, F.Cu at (-46.3, 73.9)
- added R204: 0R, Resistor_SMD:R_0402_1005Metric, F.Cu at (-32.9, 61.8)
- added R205: 0R, Resistor_SMD:R_0402_1005Metric, F.Cu at (-42.0, 70.3)
- added R206: 33R, Resistor_SMD:R_0402_1005Metric, F.Cu at (-37.7, 107.9)
- added R207: 10K, Resistor_SMD:R_0402_1005Metric, F.Cu at (-42.1, 110.0)
- added R208: 47k, Resistor_SMD:R_0402_1005Metric, F.Cu at (-39.1, 105.9)
- added R209: 33R, Resistor_SMD:R_0402_1005Metric, F.Cu at (-40.6, 107.9)
- added R21: 52.3K, Resistor_SMD:R_0402_1005Metric, F.Cu at (-25.9, 46.4)
- added R210: 33R, Resistor_SMD:R_0402_1005Metric, F.Cu at (-36.2, 100.7)
- added R211: 33R, Resistor_SMD:R_0402_1005Metric, F.Cu at (-45.0, 110.6)
- added R212: 33R, Resistor_SMD:R_0402_1005Metric, F.Cu at (-37.7, 103.4)
- added R213: 33R, Resistor_SMD:R_0402_1005Metric, F.Cu at (-42.0, 105.9)
- added R214: 33R, Resistor_SMD:R_0402_1005Metric, F.Cu at (133.1, 32.2)
- added R215: 33R, Resistor_SMD:R_0402_1005Metric, F.Cu at (133.1, 34.0)
- added R216: 33R, Resistor_SMD:R_0402_1005Metric, F.Cu at (132.8, 35.9)
- added R217: 1K, Resistor_SMD:R_0402_1005Metric, F.Cu at (-74.3, 41.1)
- added R22: 43K, Resistor_SMD:R_0402_1005Metric, F.Cu at (-20.2, 39.9)
- added R23: 33R, Resistor_SMD:R_0402_1005Metric, F.Cu at (-25.9, 44.4)
- added R24: 33R, Resistor_SMD:R_0402_1005Metric, F.Cu at (-30.3, 48.9)
- added R25: 33R, Resistor_SMD:R_0402_1005Metric, F.Cu at (-33.7, 52.3)
- added R26: 33R, Resistor_SMD:R_0402_1005Metric, F.Cu at (-37.2, 55.3)
- added R27: 33R, Resistor_SMD:R_0402_1005Metric, F.Cu at (-33.2, 49.8)
- added R28: 33R, Resistor_SMD:R_0402_1005Metric, F.Cu at (-24.5, 42.4)
- added R29: 33R, Resistor_SMD:R_0402_1005Metric, F.Cu at (-28.8, 46.8)
- added R3: 33R, Resistor_SMD:R_0402_1005Metric, F.Cu at (108.1, 68.8)
- added R30: 10K, Resistor_SMD:R_0402_1005Metric, F.Cu at (-23.1, 39.9)
- added R31: 10K, Resistor_SMD:R_0402_1005Metric, F.Cu at (-24.9, 56.8)
- added R32: 33R, Resistor_SMD:R_0402_1005Metric, F.Cu at (18.5, 11.2)
- added R33: 33R, Resistor_SMD:R_0402_1005Metric, F.Cu at (23.9, 22.5)
- added R34: 33R, Resistor_SMD:R_0402_1005Metric, F.Cu at (17.1, 11.1)
- added R35: 33R, Resistor_SMD:R_0402_1005Metric, F.Cu at (22.0, 22.3)
- added R36: 10K, Resistor_SMD:R_0402_1005Metric, F.Cu at (23.5, 16.6)
- added R37: 10K, Resistor_SMD:R_0402_1005Metric, F.Cu at (25.0, 16.6)
- added R38: 33R, Resistor_SMD:R_0402_1005Metric, F.Cu at (15.6, 11.0)
- added R39: 33R, Resistor_SMD:R_0402_1005Metric, F.Cu at (20.2, 22.8)
- added R4: 33R, Resistor_SMD:R_0402_1005Metric, F.Cu at (108.1, 70.5)
- added R40: 33R, Resistor_SMD:R_0402_1005Metric, F.Cu at (14.1, 11.4)
- added R41: 33R, Resistor_SMD:R_0402_1005Metric, F.Cu at (18.0, 22.7)
- added R42: 33R, Resistor_SMD:R_0402_1005Metric, F.Cu at (12.4, 11.5)
- added R43: 33R, Resistor_SMD:R_0402_1005Metric, F.Cu at (16.2, 22.8)
- added R44: 33R, Resistor_SMD:R_0402_1005Metric, F.Cu at (10.6, 11.4)
- added R45: 33R, Resistor_SMD:R_0402_1005Metric, F.Cu at (14.3, 22.8)
- added R46: 10K, Resistor_SMD:R_0402_1005Metric, F.Cu at (3.90, 15.8)
- added R47: 33R, Resistor_SMD:R_0402_1005Metric, F.Cu at (6.70, 23.1)
- added R48: 33R, Resistor_SMD:R_0402_1005Metric, F.Cu at (8.40, 23.0)
- added R49: 33R, Resistor_SMD:R_0402_1005Metric, F.Cu at (9.50, 23.0)
- added R5: 33R, Resistor_SMD:R_0402_1005Metric, F.Cu at (108.0, 72.2)
- added R50: 33R, Resistor_SMD:R_0402_1005Metric, F.Cu at (44.6, 85.3)
- added R51: 33R, Resistor_SMD:R_0402_1005Metric, F.Cu at (46.1, 65.2)
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Other:
- board size 102 x 148 mm -> 148 x 102 mm

Commit message: ...
Parts:
- removed R15: 33R, Resistor_SMD:R_0402_1005Metric
- J12, J13: footprint Connector_USB:USB_Micro-B_Molex-105017-0001 -> FlightComputer_Library:USB_Micro-B_TE-1981568-1
- X1: footprint Oscillator:Oscillator_SMD_Abracon_ASE-4Pin_3.2x2.5mm_HandSoldering -> Oscillator:Oscillator_SMD_Abracon_ASE-4Pin_3.2x2.5mm
- Y1: footprint Crystal:Crystal_SMD_3225-4Pin_3.2x2.5mm_HandSoldering -> Crystal:Crystal_SMD_3225-4Pin_3.2x2.5mm
- moved D8 235.1 mm to (146.5, 17.7), turned to 270 degrees
- moved R118 229.5 mm to (144.1, 16.8), turned to 180 degrees
- moved D7 229.4 mm to (146.9, 3.00), turned to 270 degrees
- moved R117 226.8 mm to (144.1, 2.20), turned to 180 degrees
- moved R217 221.6 mm to (144.1, 3.50), turned to 180 degrees
- moved R211 205.6 mm to (133.9, 9.10)
- moved R213 201.4 mm to (133.9, 7.80)
- moved C120 200.5 mm to (138.0, 13.9), turned to 180 degrees
- moved R207 200.5 mm to (133.9, 13.9), turned to 180 degrees
- moved R209 197.7 mm to (133.9, 15.1)
- moved R206 196.2 mm to (133.9, 12.7)
- moved R119 195.3 mm to (116.4, 18.3)
- moved R208 194.8 mm to (133.9, 16.3), turned to 180 degrees
- moved R212 194.6 mm to (133.9, 11.5)
- moved R129 194.3 mm to (104.3, 29.9)
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Connections:
- J1 pad 5: Net-(J1-Pad5) -> (no net)
- J11 pad 10: Net-(J11-Pad10) -> (no net)
- J11 pad 12: Net-(J11-Pad12) -> (no net)
- J11 pad 14: Net-(J11-Pad14) -> (no net)
- J11 pad 16: Net-(J11-Pad16) -> (no net)
- J11 pad 18: Net-(J11-Pad18) -> (no net)
- J11 pad 20: Net-(J11-Pad20) -> (no net)
- J11 pad 22: Net-(J11-Pad22) -> (no net)
- J11 pad 23: Net-(J11-Pad23) -> (no net)
- J11 pad 24: Net-(J11-Pad24) -> (no net)
- J11 pad 26: Net-(J11-Pad26) -> (no net)
- J11 pad 28: Net-(J11-Pad28) -> (no net)
- J11 pad 3: Net-(J11-Pad3) -> (no net)
- J11 pad 30: Net-(J11-Pad30) -> (no net)
- J11 pad 32: Net-(J11-Pad32) -> (no net)
- J11 pad 34: Net-(J11-Pad34) -> (no net)
- J11 pad 36: Net-(J11-Pad36) -> (no net)
- J11 pad 37: Net-(J11-Pad37) -> (no net)
- J11 pad 38: Net-(J11-Pad38) -> (no net)
- J11 pad 4: Net-(J11-Pad4) -> (no net)
- J11 pad 6: Net-(J11-Pad6) -> (no net)
- J11 pad 8: Net-(J11-Pad8) -> (no net)
- J13 pad 4: Net-(J13-Pad4) -> (no net)
- J2 pad 3: Net-(J2-Pad3) -> (no net)
- J2 pad 6: Net-(J2-Pad6) -> (no net)
- J2 pad 9: Net-(J2-Pad9) -> (no net)
- J6 pad 11: Net-(J6-Pad11) -> (no net)
- J6 pad 17: Net-(J6-Pad17) -> (no net)
- J6 pad 26: Net-(J6-Pad26) -> (no net)
- J6 pad 27: Net-(J6-Pad27) -> (no net)
- J6 pad 28: Net-(J6-Pad28) -> (no net)
- J6 pad 29: Net-(J6-Pad29) -> (no net)
- J6 pad 31: Net-(J6-Pad31) -> (no net)
- J6 pad 32: Net-(J6-Pad32) -> (no net)
- J6 pad 33: Net-(J6-Pad33) -> (no net)
- J6 pad 36: Net-(J6-Pad36) -> (no net)
- J6 pad 7: Net-(J6-Pad7) -> (no net)
- J7 pad 9: Net-(J7-Pad9) -> (no net)
- M1 pad 4: Net-(M1-Pad4) -> (no net)
- M2 pad 2: Net-(M2-Pad2) -> (no net)
- M3 pad 2: Net-(M3-Pad2) -> (no net)
- U10 pad 2: Net-(U10-Pad2) -> (no net)
- U3 pad 3: Net-(U3-Pad3) -> (no net)
- X1 pad 3: Net-(R15-Pad1) -> /Codec/I2S_MCLK
- Y1 pad 2: Net-(Y1-Pad2) -> (no net)
- Y1 pad 4: Net-(Y1-Pad4) -> (no net)

Commit message: ...
Parts:
- moved TP14 126.8 mm to (39.8, 39.3)
- moved TP15 126.8 mm to (39.8, 41.5)
- moved R199 125.6 mm to (83.0, 28.6), turned to 270 degrees
- moved R196 124.5 mm to (84.3, 28.5), turned to 270 degrees
- moved TP13 122.7 mm to (39.8, 52.3)
- moved C92 121.6 mm to (63.6, 25.8), turned to 270 degrees
- moved C93 117.6 mm to (83.0, 25.8), turned to 270 degrees
- moved C88 117.2 mm to (84.3, 26.3), turned to 90 degrees
- moved TP7 115.7 mm to (69.5, 23.5)
- moved R189 114.3 mm to (34.5, 47.9)
- moved R190 113.7 mm to (34.6, 46.8)
- moved C90 113.6 mm to (87.9, 40.8)
- moved R126 112.2 mm to (69.5, 28.6), turned to 90 degrees
- moved R198 112.1 mm to (78.4, 62.1), turned to 90 degrees
- moved R195 109.8 mm to (76.9, 62.2), turned to 90 degrees
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Routing:
- added copper zone on F.Cu, net GND
Other:
- copper layers 2 -> 4

Commit message: ...
Parts:
- moved J8 16.1 mm to (126.5, 3.00), turned to 270 degrees
- moved C56 7.77 mm to (118.1, 15.8), turned to 0 degrees
- moved C85 5.65 mm to (101.7, 81.4)
- moved C86 5.65 mm to (101.7, 73.0)
- moved R186 5.65 mm to (101.7, 83.4)
- moved R188 5.65 mm to (101.7, 75.5)
- moved R187 5.65 mm to (101.7, 74.3)
- moved SW10 5.65 mm to (98.2, 82.4)
- moved SW11 5.65 mm to (98.2, 74.3)
- moved R191 4.88 mm to (10.0, 68.7), turned to 270 degrees
- moved R148 4.70 mm to (19.9, 73.8)
- moved R149 4.70 mm to (19.9, 75.0)
- moved R150 3.90 mm to (10.00, 74.4)
- moved R151 3.90 mm to (11.3, 74.4)
- moved R152 3.90 mm to (12.5, 74.4)
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Routing:
- net VCC_PERIH: track 0.00 -> 25.5 mm
- net Net-(R57-Pad1): track 0.00 -> 5.41 mm
- net Net-(R55-Pad1): track 0.00 -> 5.33 mm
- net Net-(R53-Pad1): track 0.00 -> 5.24 mm
- net Net-(R51-Pad1): track 0.00 -> 5.16 mm
- net Net-(R50-Pad2): track 0.00 -> 5.08 mm
- net Net-(R74-Pad1): track 0.00 -> 5.08 mm
- net Net-(R56-Pad2): track 0.00 -> 5.08 mm
- net Net-(R64-Pad2): track 0.00 -> 5.00 mm
- net Net-(R58-Pad2): track 0.00 -> 5.00 mm
- net Net-(R86-Pad1): track 0.00 -> 5.00 mm
- net Net-(R52-Pad2): track 0.00 -> 4.91 mm
- net Net-(R85-Pad1): track 0.00 -> 4.91 mm
- net Net-(R60-Pad2): track 0.00 -> 4.83 mm
- net Net-(R54-Pad2): track 0.00 -> 4.83 mm
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
Commit message: ...
Parts:
- moved C93 19.5 mm to (63.5, 25.7)
- moved C92 19.4 mm to (83.0, 25.6)
- moved C56 8.32 mm to (111.3, 11.0), turned to 180 degrees
- moved R138 5.69 mm to (56.3, 14.5), turned to 90 degrees
- moved R194 4.72 mm to (51.2, 34.7)
- moved L7 4.50 mm to (128.5, 43.7)
- moved R137 3.72 mm to (54.0, 16.7), turned to 270 degrees
- moved R140 3.21 mm to (54.0, 18.8), turned to 90 degrees
- moved R139 2.95 mm to (53.0, 18.8), turned to 90 degrees
- moved D9 2.59 mm to (53.4, 14.1)
- moved R203 2.44 mm to (51.3, 44.3)
- moved R206 2.40 mm to (133.9, 15.1)
- moved R207 2.40 mm to (133.9, 16.3)
- moved R208 2.40 mm to (133.9, 13.9)
- moved R209 2.40 mm to (133.9, 12.7)
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Connections:
- J1 pad 5: (no net) -> Net-(J1-Pad5)
- J11 pad 10: (no net) -> Net-(J11-Pad10)
- J11 pad 12: (no net) -> Net-(J11-Pad12)
- J11 pad 14: (no net) -> Net-(J11-Pad14)
- J11 pad 16: (no net) -> Net-(J11-Pad16)
- J11 pad 18: (no net) -> Net-(J11-Pad18)
- J11 pad 20: (no net) -> Net-(J11-Pad20)
- J11 pad 22: (no net) -> Net-(J11-Pad22)
- J11 pad 23: (no net) -> Net-(J11-Pad23)
- J11 pad 24: (no net) -> Net-(J11-Pad24)
- J11 pad 26: (no net) -> Net-(J11-Pad26)
- J11 pad 28: (no net) -> Net-(J11-Pad28)
- J11 pad 3: (no net) -> Net-(J11-Pad3)
- J11 pad 30: (no net) -> Net-(J11-Pad30)
- J11 pad 32: (no net) -> Net-(J11-Pad32)
- J11 pad 34: (no net) -> Net-(J11-Pad34)
- J11 pad 36: (no net) -> Net-(J11-Pad36)
- J11 pad 37: (no net) -> Net-(J11-Pad37)
- J11 pad 38: (no net) -> Net-(J11-Pad38)
- J11 pad 4: (no net) -> Net-(J11-Pad4)
- J11 pad 6: (no net) -> Net-(J11-Pad6)
- J11 pad 8: (no net) -> Net-(J11-Pad8)
- J13 pad 4: (no net) -> Net-(J13-Pad4)
- J2 pad 3: (no net) -> Net-(J2-Pad3)
- J2 pad 6: (no net) -> Net-(J2-Pad6)
- J2 pad 9: (no net) -> Net-(J2-Pad9)
- J6 pad 11: (no net) -> Net-(J6-Pad11)
- J6 pad 17: (no net) -> Net-(J6-Pad17)
- J6 pad 26: (no net) -> Net-(J6-Pad26)
- J6 pad 27: (no net) -> Net-(J6-Pad27)
- J6 pad 28: (no net) -> Net-(J6-Pad28)
- J6 pad 29: (no net) -> Net-(J6-Pad29)
- J6 pad 31: (no net) -> Net-(J6-Pad31)
- J6 pad 32: (no net) -> Net-(J6-Pad32)
- J6 pad 33: (no net) -> Net-(J6-Pad33)
- J6 pad 36: (no net) -> Net-(J6-Pad36)
- J6 pad 7: (no net) -> Net-(J6-Pad7)
- J7 pad 9: (no net) -> Net-(J7-Pad9)
- M1 pad 4: (no net) -> Net-(M1-Pad4)
- M2 pad 2: (no net) -> Net-(M2-Pad2)
- M3 pad 2: (no net) -> Net-(M3-Pad2)
- U10 pad 2: (no net) -> Net-(U10-Pad2)
- U13 pad 100: GNDS -> GND
- U13 pad 106: GNDS -> GND
- U13 pad 112: GNDS -> GND
- U13 pad 119: GNDS -> GND
- U13 pad 12: GNDS -> GND
- U13 pad 134: GNDS -> GND
- U13 pad 137: GNDS -> GND
- U13 pad 151: GNDS -> GND
- U13 pad 159: GNDS -> GND
- U13 pad 173: GNDS -> GND
- U13 pad 24: GNDS -> GND
- U13 pad 45: GNDS -> GND
- U13 pad 47: GNDS -> GND
- U13 pad 6: GNDS -> GND
- U13 pad 64: GNDS -> GND
- U13 pad 70: GNDS -> GND
- U13 pad 81: GNDS -> GND
- U13 pad 83: GNDS -> GND
- U13 pad 93: GNDS -> GND
- U3 pad 3: (no net) -> Net-(U3-Pad3)
- Y1 pad 2: (no net) -> Net-(Y1-Pad2)
- Y1 pad 4: (no net) -> Net-(Y1-Pad4)
Routing:
- net VCC_3V3: track 0.00 -> 169.2 mm, vias 0 -> 11
- net Net-(R9-Pad1): track 0.00 -> 66.5 mm, vias 0 -> 6
- net Net-(C9-Pad1): track 0.00 -> 59.5 mm, vias 0 -> 4
- net /Codec/I2C_SDA: track 0.00 -> 56.5 mm, vias 0 -> 1
- net /Codec/I2C_SCL: track 0.00 -> 51.9 mm, vias 0 -> 1
- net Net-(C8-Pad1): track 0.00 -> 48.8 mm, vias 0 -> 2
- net /Codec/I2S_SCLK: track 0.00 -> 42.8 mm, vias 0 -> 2
- net /Codec/RADIO_L: track 0.00 -> 41.5 mm, vias 0 -> 2
- net (no net): track 0.00 -> 40.6 mm
- net /Codec/RADIO_R: track 0.00 -> 38.5 mm, vias 0 -> 2
- net Net-(L3-Pad1): track 0.00 -> 37.8 mm, vias 0 -> 2
- net /Raspberry/SDIO_DAT2: track 0.00 -> 34.8 mm, vias 0 -> 2
- net Net-(L4-Pad1): track 0.00 -> 34.7 mm, vias 0 -> 2
- net VCC_5V: track 0.00 -> 34.2 mm, vias 0 -> 4
- net GND: track 0.00 -> 34.2 mm, vias 0 -> 19
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- added copper zone on In1.Cu, net GND
- added copper zone on In2.Cu, net VCC_5V

Commit message: ...
Parts:
- moved C121 18.0 mm to (137.6, 13.5)
- moved R214 18.0 mm to (133.5, 10.4)
- moved R215 18.0 mm to (133.5, 9.20)
- moved R216 18.0 mm to (133.5, 11.6)
- moved U16 18.0 mm to (137.6, 10.4)
- moved J12 18.0 mm to (146.0, 28.1)
- moved J13 18.0 mm to (146.0, 10.2)
- moved C120 17.5 mm to (140.1, 33.0)
- moved R206 17.5 mm to (133.5, 32.6)
- moved R208 17.5 mm to (133.5, 31.4)
- moved R209 17.5 mm to (133.5, 30.2)
- moved R210 17.5 mm to (133.5, 27.8)
- moved R211 17.5 mm to (133.5, 26.6)
- moved R212 17.5 mm to (133.5, 29.0)
- moved R213 17.5 mm to (133.5, 25.3)
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Routing:
- net Net-(J12-Pad3): track 4.43 -> 6.97 mm
- net Net-(J12-Pad4): track 9.67 -> 11.3 mm
- net GND: track 34.2 -> 33.6 mm, vias 19 -> 18
