File: hw/rev1/FlightComputer/FlightComputer.kicad_pcb (KiCad board)
At the start: 4 copper layers, 148 x 102 mm, 372 parts, among them J1 Conn_01x10, J11 Conn_02x20_Odd_Even, J12 USB_B_Micro, J13 USB_B_Micro, J2 Conn_01x10, J4 Conn_01x01, J5 ED060SC7_EPD, J6 RPI_Connector, J7 Micro_SD_Card, J8 Conn_01x02, M1 TEA5767_Radio_Module, M2 GY-91, M3 GY-86, SW10 SW_Push, SW11 SW_Push, U1 WM8960, U10 TPS61090, U11 TPS22917DBV, U13 STM32H745IIT, U14 STMPS2151STR, U15 USBLC6-2SC6, U16 USBLC6-2SC6, U2 TPS65186, U3 MT25QL512ABB8ESF, U4 MT48LC16M16A2P, U5 MAX809TTRG, U6 XC6220B331MR-G, U7 MCP73871, U8 XC6220B331MR-G, X1 24MHz, Y1 25MHz

Commit message: ...
Parts:
- moved R21 9.33 mm to (15.5, 39.3)
- moved C24 9.09 mm to (26.1, 41.2), turned to 90 degrees
- moved R19 6.99 mm to (14.2, 39.3)
- moved R18 6.89 mm to (13.1, 39.3)
- moved R187 6.80 mm to (97.3, 69.1), turned to 90 degrees
- moved R20 6.65 mm to (16.6, 39.3), turned to 90 degrees
- moved R123 6.64 mm to (94.7, 51.7), turned to 0 degrees
- moved C30 6.22 mm to (16.1, 37.7), turned to 180 degrees
- moved R122 5.91 mm to (94.7, 52.9)
- moved D1 5.19 mm to (8.20, 44.8), turned to 90 degrees
- moved L9 4.70 mm to (31.1, 38.4)
- moved C29 4.68 mm to (13.6, 37.7), turned to 180 degrees
- moved D2 4.62 mm to (26.1, 37.6), turned to 270 degrees
- moved R189 4.25 mm to (38.7, 48.8), turned to 90 degrees
- moved R190 4.14 mm to (38.7, 46.8), turned to 270 degrees
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Connections:
- J1 pad 5: Net-(J1-Pad5) -> (no net)
- J11 pad 10: Net-(J11-Pad10) -> (no net)
- J11 pad 11: KEY_DOWN -> G_KEY_DOWN
- J11 pad 12: Net-(J11-Pad12) -> (no net)
- J11 pad 13: KEY_ENTER -> G_KEY_ENTER
- J11 pad 14: Net-(J11-Pad14) -> (no net)
- J11 pad 15: KEY_MENU -> G_KEY_MENU
- J11 pad 16: Net-(J11-Pad16) -> (no net)
- J11 pad 17: KEY_ESCAPE -> G_KEY_ESCAPE
- J11 pad 18: Net-(J11-Pad18) -> (no net)
- J11 pad 19: KEY_FUNC1 -> G_KEY_FUNC1
- J11 pad 20: Net-(J11-Pad20) -> (no net)
- J11 pad 21: KEY_FUNC2 -> G_KEY_FUNC2
- J11 pad 22: Net-(J11-Pad22) -> (no net)
- J11 pad 23: Net-(J11-Pad23) -> (no net)
- J11 pad 24: Net-(J11-Pad24) -> (no net)
- J11 pad 26: Net-(J11-Pad26) -> (no net)
- J11 pad 28: Net-(J11-Pad28) -> (no net)
- J11 pad 3: Net-(J11-Pad3) -> (no net)
- J11 pad 30: Net-(J11-Pad30) -> (no net)
- J11 pad 32: Net-(J11-Pad32) -> (no net)
- J11 pad 34: Net-(J11-Pad34) -> (no net)
- J11 pad 36: Net-(J11-Pad36) -> (no net)
- J11 pad 37: Net-(J11-Pad37) -> (no net)
- J11 pad 38: Net-(J11-Pad38) -> (no net)
- J11 pad 4: Net-(J11-Pad4) -> (no net)
- J11 pad 5: KEY_LEFT -> G_KEY_LEFT
- J11 pad 6: Net-(J11-Pad6) -> (no net)
- J11 pad 7: KEY_RIGHT -> G_KEY_RIGHT
- J11 pad 8: Net-(J11-Pad8) -> (no net)
- J11 pad 9: KEY_UP -> G_KEY_UP
- J13 pad 4: Net-(J13-Pad4) -> (no net)
- J2 pad 3: Net-(J2-Pad3) -> (no net)
- J2 pad 6: Net-(J2-Pad6) -> (no net)
- J2 pad 9: Net-(J2-Pad9) -> (no net)
- J6 pad 11: Net-(J6-Pad11) -> (no net)
- J6 pad 17: Net-(J6-Pad17) -> (no net)
- J6 pad 26: Net-(J6-Pad26) -> (no net)
- J6 pad 27: Net-(J6-Pad27) -> (no net)
- J6 pad 28: Net-(J6-Pad28) -> (no net)
- J6 pad 29: Net-(J6-Pad29) -> (no net)
- J6 pad 31: Net-(J6-Pad31) -> (no net)
- J6 pad 32: Net-(J6-Pad32) -> (no net)
- J6 pad 33: Net-(J6-Pad33) -> (no net)
- J6 pad 36: Net-(J6-Pad36) -> (no net)
- J6 pad 7: Net-(J6-Pad7) -> (no net)
- J7 pad 9: Net-(J7-Pad9) -> (no net)
- M1 pad 4: Net-(M1-Pad4) -> (no net)
- M2 pad 2: Net-(M2-Pad2) -> (no net)
- M3 pad 2: Net-(M3-Pad2) -> (no net)
- R157 pad 1: KEY_UP -> G_KEY_UP
- R157 pad 2: KEY_UP -> /KEYBOARD/KEY_UP
- R158 pad 1: KEY_DOWN -> G_KEY_DOWN
- R158 pad 2: KEY_DOWN -> /KEYBOARD/KEY_DOWN
- R159 pad 1: KEY_LEFT -> G_KEY_LEFT
- R159 pad 2: KEY_LEFT -> /KEYBOARD/KEY_LEFT
- R160 pad 1: KEY_RIGHT -> G_KEY_RIGHT
- R160 pad 2: KEY_RIGHT -> /KEYBOARD/KEY_RIGHT
- R165 pad 1: KEY_ENTER -> G_KEY_ENTER
- R165 pad 2: KEY_ENTER -> /KEYBOARD/KEY_ENTER
- R166 pad 1: KEY_ESCAPE -> G_KEY_ESCAPE
- R166 pad 2: KEY_ESCAPE -> /KEYBOARD/KEY_ESCAPE
- R167 pad 1: KEY_FUNC1 -> G_KEY_FUNC1
- R167 pad 2: KEY_FUNC1 -> /KEYBOARD/KEY_FUNC1
- R168 pad 1: KEY_FUNC2 -> G_KEY_FUNC2
- R168 pad 2: KEY_FUNC2 -> /KEYBOARD/KEY_FUNC2
- R173 pad 1: KEY_MENU -> G_KEY_MENU
- R173 pad 2: KEY_MENU -> /KEYBOARD/KEY_MENU
- U10 pad 2: Net-(U10-Pad2) -> (no net)
- U13 pad 122: KEY_UP -> /KEYBOARD/KEY_UP
- U13 pad 123: KEY_DOWN -> /KEYBOARD/KEY_DOWN
- U13 pad 124: KEY_FUNC1 -> /KEYBOARD/KEY_FUNC1
- U13 pad 125: KEY_FUNC2 -> /KEYBOARD/KEY_FUNC2
- U13 pad 41: KEY_ENTER -> /KEYBOARD/KEY_ENTER
- U13 pad 42: KEY_MENU -> /KEYBOARD/KEY_MENU
- U13 pad 53: KEY_LEFT -> /KEYBOARD/KEY_LEFT
- U13 pad 54: KEY_RIGHT -> /KEYBOARD/KEY_RIGHT
- U13 pad 9: KEY_ESCAPE -> /KEYBOARD/KEY_ESCAPE
- U3 pad 3: Net-(U3-Pad3) -> (no net)
- Y1 pad 2: Net-(Y1-Pad2) -> (no net)
- Y1 pad 4: Net-(Y1-Pad4) -> (no net)
Routing:
- net VCC_BAT: track 0.00 -> 134.8 mm
- net VCC_EINK: track 0.00 -> 134.6 mm, vias 0 -> 6
- net GND: track 33.6 -> 85.3 mm, vias 18 -> 31
- net -15V: track 0.00 -> 49.5 mm, vias 0 -> 2
- net /EINK-PMIC/VCOM: track 0.00 -> 48.6 mm, vias 0 -> 2
- net +15V: track 0.00 -> 45.5 mm, vias 0 -> 2
- net (no net): track 40.6 -> 0.20 mm
- net Net-(C24-Pad2): track 0.00 -> 38.2 mm, vias 0 -> 2
- net VCC_PERIH: track 25.5 -> 54.7 mm, vias 0 -> 8
- net Net-(M2-Pad4): track 0.00 -> 27.0 mm
- net -20V: track 0.00 -> 26.2 mm, vias 0 -> 2
- net +22V: track 0.00 -> 25.1 mm, vias 0 -> 2
- net Net-(M2-Pad5): track 0.00 -> 22.2 mm, vias 0 -> 2
- net VCC_BAT+: track 0.00 -> 21.8 mm, vias 0 -> 3
- net Net-(M3-Pad4): track 0.00 -> 21.6 mm
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- added copper zone on In1.Cu, net GNDS
- added copper zone on In2.Cu, net VCC_BAT+
- added copper zone on In2.Cu, net VCC_MCU
- added copper zone on In2.Cu, net VCC_PERIH
Other:
- net class Default: via_dia 0.8 -> 0.6; via_drill 0.4 -> 0.3
- net class Power added: clearance 0.2, trace_width 0.4, via_dia 0.8, via_drill 0.4
- rule via_min_drill: 0.3 -> 0.2
