File: hw/rev1/FlightComputer-Extra/FlightComputer-Extra.kicad_pcb (KiCad board)
At the start: 2 copper layers, 128 x 19.8 mm, 0 parts

Commit message: ...
Parts:
- added C1: 22pF, Capacitor_SMD:C_0402_1005Metric, F.Cu at (82.6, 98.2)
- added C2: 0.1uF, Capacitor_SMD:C_0402_1005Metric, F.Cu at (128.8, 97.5)
- added J1: SJ-43617-SMT, FlightComputer_Library:SJ-43617-SMT, F.Cu at (149.0, 82.6)
- added J2: Conn_01x10, Connector_PinHeader_2.54mm:PinHeader_1x10_P2.54mm_Vertical, F.Cu at (158.1, 99.9)
- added J3: Conn_01x10, Connector_PinHeader_2.54mm:PinHeader_1x10_P2.54mm_Vertical, F.Cu at (95.9, 99.3)
- added J4: IPEX_IPX, FlightComputer_Library:IPEX-IPX, F.Cu at (104.3, 86.6)
- added J5: Conn_DEBUG, Connector_Molex:Molex_SPOX_5268-04A_1x04_P2.50mm_Horizontal, F.Cu at (130.8, 89.6)
- added L1: 33nH, Inductor_SMD:L_0402_1005Metric, F.Cu at (109.7, 86.5)
- added LS1: Speaker, FlightComputer_Library:SM150808-8, F.Cu at (194.4, 88.8)
- added LS2: Speaker, FlightComputer_Library:SM150808-8, F.Cu at (169.8, 88.6)
- added R1: 100K, Resistor_SMD:R_0402_1005Metric, F.Cu at (157.4, 86.0)
- added R2: 33R, Resistor_SMD:R_0402_1005Metric, F.Cu at (97.5, 95.8)
- added R3: 33R, Resistor_SMD:R_0402_1005Metric, F.Cu at (90.7, 96.1)
- added R4: 33R, Resistor_SMD:R_0402_1005Metric, F.Cu at (117.2, 94.2)
- added R5: 33R, Resistor_SMD:R_0402_1005Metric, F.Cu at (114.2, 94.6)
- added TP1: SCL, TestPoint:TestPoint_Pad_D1.0mm, F.Cu at (79.0, 93.3)
- added TP2: SDA, TestPoint:TestPoint_Pad_D1.0mm, F.Cu at (79.1, 90.6)
- added TP3: nRST, TestPoint:TestPoint_Pad_D1.0mm, F.Cu at (99.0, 84.2)
- added TP4: WAKEUP, TestPoint:TestPoint_Pad_D1.0mm, F.Cu at (99.2, 88.0)
- added TP5: 1PPS, TestPoint:TestPoint_Pad_D1.0mm, F.Cu at (99.8, 92.1)
- added U1: Teseo-LIV3F, FlightComputer_Library:Teseo-LIV3F, F.Cu at (90.5, 88.4)

Commit message: ...
Parts:
- moved C2 27.4 mm to (103.7, 86.7), turned to 180 degrees
- moved J4 24.1 mm to (80.2, 85.7), turned to 90 degrees
- moved LS1 23.1 mm to (171.3, 88.1)
- moved L1 22.8 mm to (86.9, 86.1), turned to 90 degrees
- moved LS2 22.4 mm to (192.2, 88.2)
- moved R3 12.8 mm to (103.5, 95.8), turned to 90 degrees
- moved C1 11.9 mm to (85.3, 86.7)
- moved R2 8.60 mm to (106.1, 95.8), turned to 90 degrees
- moved R4 6.31 mm to (111.1, 95.8), turned to 270 degrees
- moved TP3 4.83 mm to (103.8, 84.5)
- moved TP4 4.70 mm to (103.8, 88.9)
- moved U1 4.16 mm to (94.6, 88.9)
- moved TP5 4.09 mm to (103.8, 91.2)
- moved TP1 1.56 mm to (80.0, 94.5)
- moved R5 1.30 mm to (113.7, 95.8), turned to 270 degrees
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Routing:
- net VCC_PERIH: track 0.00 -> 63.8 mm
- net /HP_DETECT: track 0.00 -> 42.2 mm, vias 0 -> 2
- net /HP_RIGHT: track 0.00 -> 33.5 mm, vias 0 -> 2
- net /SPK_RP: track 0.00 -> 29.5 mm, vias 0 -> 2
- net /HP_LEFT: track 0.00 -> 22.9 mm
- net Net-(J5-Pad3): track 0.00 -> 22.2 mm
- net Net-(J5-Pad2): track 0.00 -> 22.2 mm, vias 0 -> 1
- net /SPK_LN: track 0.00 -> 15.7 mm, vias 0 -> 1
- net VCC_3V3: track 0.00 -> 15.7 mm, vias 0 -> 1
- net /SPK_LP: track 0.00 -> 13.8 mm
- net GND: track 0.00 -> 13.6 mm
- net /SPK_RN: track 0.00 -> 13.0 mm
- net Net-(TP1-Pad1): track 0.00 -> 11.0 mm
- net Net-(TP2-Pad1): track 0.00 -> 10.1 mm
- net Net-(R2-Pad2): track 0.00 -> 9.37 mm, vias 0 -> 2
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- added copper zone on B.Cu, net GND
- added copper zone on F.Cu, net GND

Commit message: ...
Parts:
- moved J5 9.43 mm to (121.4, 88.8)
- moved J3 4.86 mm to (99.8, 96.4)
- moved U1 4.73 mm to (90.0, 87.8)
- moved R3 4.57 mm to (107.5, 93.6)
- moved R2 4.48 mm to (110.0, 93.6)
- moved R4 4.43 mm to (115.0, 93.7)
- moved R5 4.43 mm to (117.6, 93.7)
- moved R1 3.63 mm to (157.2, 89.3), turned to 90 degrees
- moved J2 3.52 mm to (157.2, 96.5)
- moved LS1 2.16 mm to (173.4, 87.6)
- moved LS2 0.59 mm to (192.4, 87.6)
- moved J1 0.54 mm to (148.8, 82.1)
Routing:
- net VCC_PERIH: track 63.8 -> 0.00 mm
- net /HP_DETECT: track 42.2 -> 0.00 mm, vias 2 -> 0
- net /HP_RIGHT: track 33.5 -> 0.00 mm, vias 2 -> 0
- net /SPK_RP: track 29.5 -> 0.00 mm, vias 2 -> 0
- net /HP_LEFT: track 22.9 -> 0.00 mm
- net Net-(J5-Pad3): track 22.2 -> 0.00 mm
- net Net-(J5-Pad2): track 22.2 -> 0.00 mm, vias 1 -> 0
- net /SPK_LN: track 15.7 -> 0.00 mm, vias 1 -> 0
- net VCC_3V3: track 15.7 -> 0.00 mm, vias 1 -> 0
- net /SPK_LP: track 13.8 -> 0.00 mm
- net GND: track 13.6 -> 0.00 mm
- net /SPK_RN: track 13.0 -> 0.00 mm
- net Net-(TP1-Pad1): track 11.0 -> 0.00 mm
- net Net-(TP2-Pad1): track 10.1 -> 0.00 mm
- net Net-(R2-Pad2): track 9.37 -> 0.00 mm, vias 2 -> 0
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- removed copper zone on B.Cu, net GND
- removed copper zone on F.Cu, net GND
Other:
- board size 128 x 19.8 mm -> 128 x 16.9 mm

Commit message: pcb dimension
Parts:
- added C3: 1uF, Capacitor_SMD:C_0402_1005Metric, F.Cu at (98.9, 85.9)
- moved R1 6.57 mm to (152.0, 85.2), turned to 180 degrees
- moved C2 4.82 mm to (98.9, 87.0)
- moved J1 4.00 mm to (144.8, 82.1)
- moved L1 3.27 mm to (83.6, 86.4)
- moved C1 2.54 mm to (83.1, 88.0)
- moved U1 1.76 mm to (91.1, 89.2)
- moved TP1 1.20 mm to (79.2, 93.6)
- moved TP5 0.96 mm to (103.5, 90.3)
- moved TP2 0.94 mm to (79.2, 91.4)
- moved J5 0.90 mm to (120.5, 88.8)
- moved J4 0.87 mm to (79.3, 85.9)
- moved TP4 0.77 mm to (103.5, 88.2)
- moved TP3 0.43 mm to (103.5, 84.8)
- moved LS1 0.30 mm to (173.4, 87.9)
- moved LS2 0.30 mm to (192.4, 87.9)
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Connections:
- J1 pad 1: GND -> GNDA
- J2 pad 10: GND -> GNDA
Routing:
- net /HP_DETECT: track 0.00 -> 55.0 mm, vias 0 -> 1
- net VCC_PERIH: track 0.00 -> 54.0 mm, vias 0 -> 1
- net /HP_RIGHT: track 0.00 -> 39.7 mm, vias 0 -> 1
- net /SPK_RP: track 0.00 -> 34.5 mm, vias 0 -> 1
- net /HP_LEFT: track 0.00 -> 29.6 mm, vias 0 -> 1
- net /SPK_RN: track 0.00 -> 16.2 mm, vias 0 -> 1
- net Net-(R2-Pad2): track 0.00 -> 15.5 mm, vias 0 -> 2
- net VCC_3V3: track 0.00 -> 15.4 mm
- net /SPK_LP: track 0.00 -> 13.6 mm, vias 0 -> 1
- net Net-(R3-Pad2): track 0.00 -> 12.4 mm
- net /SPK_LN: track 0.00 -> 9.41 mm
- net Net-(TP4-Pad1): track 0.00 -> 8.21 mm
- net Net-(TP5-Pad1): track 0.00 -> 7.80 mm
- net Net-(TP3-Pad1): track 0.00 -> 7.80 mm
- net Net-(TP1-Pad1): track 0.00 -> 7.76 mm
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- added copper zone on F.Cu, net GND
- added copper zone on F.Cu, net GNDA
Other:
- outline, holes or cut-outs redrawn

Commit message: ...
Other:
- board text added: "1PPS"
- board text added: "DBG/PROG Gnd,Tx,Rx,Vcc"
- board text added: "SCL"
- board text added: "SDA"
- board text added: "WAKEUP"
- board text added: "nRST"

Commit message: ...
Parts:
- moved LS1 0.07 mm to (173.5, 87.9)
Routing:
- net /SPK_RN: track 16.2 -> 15.5 mm
- net /SPK_LP: track 13.6 -> 14.2 mm
