File: hw/rev1/FlightComputer-Extra/FlightComputer-Extra.kicad_pcb (KiCad board)
At the start: 2 copper layers, 128 x 16.9 mm, 22 parts, among them J1 SJ-43617-SMT, J2 Conn_01x10, J3 Conn_01x10, J4 IPEX_IPX, J5 Conn_DEBUG, U1 Teseo-LIV3F

Commit message: gerber
Parts:
- added G***: LOGO, FlightComputer_Library:LOGO-FC, B.Cu at (174.8, 89.8)

Commit message: gerber final
Parts:
- C1, C2, C3: footprint Capacitor_SMD:C_0402_1005Metric -> FlightComputer_Library:C_0402_1005Metric_Pad0.74x0.62mm_HandSolder
- R1, R2, R3, R4, R5: footprint Resistor_SMD:R_0402_1005Metric -> FlightComputer_Library:R_0402_1005Metric_Pad0.72x0.64mm_HandSolder
- moved R2 0.20 mm to (110.0, 93.3)
- moved R3 0.20 mm to (107.4, 93.3)
- moved L1 0.08 mm to (83.7, 86.4)
Routing:
- net /HP_RIGHT: track 39.7 -> 42.3 mm
