File: hw/rev1/FlightComputer-Keypad/FlightComputer-Keypad.kicad_pcb (KiCad board)
At the start: 2 copper layers, 47 parts, among them J1 Conn_02x20_Odd_Even, J2 Conn_02x10_Odd_Even, SW1 SW_Push, SW2 SW_Push, SW3 SW_Push, SW4 SW_Push, SW5 SW_Push, SW6 SW_Push, SW7 SW_Push, SW8 SW_Push, SW9 SW_Push

Commit message: ...
Parts:
- moved J1 84.9 mm to (126.3, 106.8), turned to 90 degrees
Other:
- board outline added: 148 x 42 mm

Commit message: ...
Parts:
- J1: footprint Connector_PinSocket_2.54mm:PinSocket_2x20_P2.54mm_Vertical -> Connector_PinHeader_2.54mm:PinHeader_2x20_P2.54mm_Vertical
- SW1, SW2, SW3, SW4, SW5, SW6, SW7, SW8, SW9: footprint FlightComputer_Library:SW_SPST_PTS647 -> FlightComputer_Library:SW-SPST-PTS647
- moved R13 151.6 mm to (201.2, 106.0)
- moved C9 148.9 mm to (201.3, 90.5)
- moved C8 147.6 mm to (201.2, 103.2)
- moved R18 146.8 mm to (201.3, 91.9), turned to 180 degrees
- moved R14 145.6 mm to (201.3, 93.3)
- moved R17 145.3 mm to (201.2, 104.6), turned to 180 degrees
- moved SW9 143.0 mm to (195.7, 91.9)
- moved R26 136.5 mm to (181.4, 89.5), turned to 90 degrees
- moved SW8 132.3 mm to (195.7, 104.6)
- moved R1 131.0 mm to (149.4, 108.5)
- moved R20 123.3 mm to (164.7, 89.5), turned to 270 degrees
- moved R25 122.8 mm to (178.8, 89.5), turned to 90 degrees
- moved J2 122.8 mm to (163.6, 85.8), turned to 90 degrees
- moved R21 121.9 mm to (166.1, 89.5), turned to 90 degrees
- moved R22 121.7 mm to (168.7, 89.5), turned to 90 degrees
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Connections:
- J1 pad 10: /KEY_DOWN -> /KEY_UP
- J1 pad 11: /KEY_POWER -> /KEY_DOWN
- J1 pad 12: /KEY_POWER -> /KEY_DOWN
- J1 pad 15: /KEY_ESCAPE -> /KEY_MENU
- J1 pad 16: /KEY_ESCAPE -> /KEY_MENU
- J1 pad 17: /KEY_FUNC1 -> /KEY_ESCAPE
- J1 pad 18: /KEY_FUNC1 -> /KEY_ESCAPE
- J1 pad 19: /KEY_FUNC2 -> /KEY_FUNC1
- J1 pad 20: /KEY_FUNC2 -> /KEY_FUNC1
- J1 pad 22: Net-(J1-Pad22) -> /KEY_FUNC2
- J1 pad 26: Net-(J1-Pad26) -> /TRST
- J1 pad 27: /TRST -> /TDI
- J1 pad 28: /TRST -> /TDI
- J1 pad 29: /TDI -> /TMS
- J1 pad 3: /KEY_LEFT -> Net-(J1-Pad3)
- J1 pad 30: /TDI -> /TMS
- J1 pad 31: /TMS -> /TCLK
- J1 pad 32: /TMS -> /TCLK
- J1 pad 33: /TCLK -> /TDO
- J1 pad 34: /TCLK -> /TDO
- J1 pad 35: /TDO -> /nRESET
- J1 pad 36: /TDO -> /nRESET
- J1 pad 37: /nRESET -> Net-(J1-Pad37)
- J1 pad 38: /nRESET -> Net-(J1-Pad37)
- J1 pad 4: /KEY_LEFT -> Net-(J1-Pad3)
- J1 pad 5: /KEY_RIGHT -> /KEY_LEFT
- J1 pad 6: /KEY_RIGHT -> /KEY_LEFT
- J1 pad 7: /KEY_UP -> /KEY_RIGHT
- J1 pad 8: /KEY_UP -> /KEY_RIGHT
- J1 pad 9: /KEY_DOWN -> /KEY_UP
Routing:
- net /KEY_FUNC2: track 0.00 -> 82.9 mm, vias 0 -> 2
- net /KEY_FUNC1: track 0.00 -> 68.7 mm, vias 0 -> 2
- net /KEY_ESCAPE: track 0.00 -> 65.4 mm, vias 0 -> 2
- net /KEY_LEFT: track 0.00 -> 54.4 mm, vias 0 -> 2
- net /KEY_ENTER: track 0.00 -> 48.9 mm, vias 0 -> 2
- net /KEY_DOWN: track 0.00 -> 44.7 mm, vias 0 -> 2
- net /TDI: track 0.00 -> 38.2 mm
- net /TRST: track 0.00 -> 37.2 mm
- net /nRESET: track 0.00 -> 34.6 mm
- net /TDO: track 0.00 -> 34.6 mm
- net /TMS: track 0.00 -> 33.6 mm
- net /TCLK: track 0.00 -> 33.1 mm
- net /KEY_UP: track 0.00 -> 28.3 mm, vias 0 -> 2
- net /KEY_RIGHT: track 0.00 -> 27.5 mm, vias 0 -> 2
- net GND: track 0.00 -> 25.8 mm, vias 0 -> 2
- added copper zone on F.Cu, net GND
- added copper zone on B.Cu, net VCC_MCU
Other:
- outline, holes or cut-outs redrawn

Commit message: ...
Parts:
- R19, R20, R27: moved to B.Cu
- moved R19 6.23 mm to (161.2, 88.9), turned to 0 degrees
- moved R20 3.55 mm to (161.2, 90.1), turned to 0 degrees
- moved J2 2.93 mm to (160.7, 86.2)
- moved R21 2.90 mm to (163.2, 89.5)
- moved R24 2.90 mm to (170.9, 89.5)
- moved R25 2.90 mm to (175.9, 89.5)
- moved R26 2.90 mm to (178.5, 89.5)
- moved R27 2.90 mm to (169.6, 89.5)
- moved R22 2.90 mm to (165.8, 89.5)
- moved R23 2.90 mm to (168.3, 89.5)
- moved J1 0.98 mm to (119.8, 120.6)
- moved C8 0.41 mm to (201.1, 102.8)
- moved C7 0.40 mm to (97.5, 90.3)
- moved C5 0.30 mm to (149.3, 96.5)
- moved R11 0.30 mm to (97.5, 106.0)
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Connections:
- J1 pad 21: Net-(J1-Pad21) -> /KEY_FUNC2
- J1 pad 25: Net-(J1-Pad25) -> /TRST
- J1 pad 38: Net-(J1-Pad37) -> Net-(J1-Pad38)
- J1 pad 4: Net-(J1-Pad3) -> Net-(J1-Pad4)
- SW5 pad 1: VCC_MCU -> Net-(C5-Pad1)
- SW5 pad 2: Net-(C5-Pad1) -> VCC_MCU
Routing:
- net VCC_MCU: track 0.00 -> 279.1 mm, vias 0 -> 10
- net GND: track 25.8 -> 17.8 mm
- net /TDI: track 38.2 -> 45.8 mm, vias 0 -> 1
- net Net-(C3-Pad1): track 0.00 -> 5.52 mm
- net Net-(C9-Pad1): track 0.00 -> 5.42 mm
- net Net-(C8-Pad1): track 0.00 -> 5.42 mm
- net Net-(C4-Pad1): track 0.00 -> 5.42 mm
- net Net-(C1-Pad1): track 0.00 -> 5.42 mm
- net /TCLK: track 33.1 -> 38.4 mm, vias 0 -> 1
- net Net-(C5-Pad1): track 0.00 -> 5.32 mm
- net Net-(C7-Pad1): track 0.00 -> 5.31 mm
- net Net-(C6-Pad1): track 0.00 -> 5.31 mm
- net /KEY_FUNC2: track 82.9 -> 88.0 mm
- net Net-(C2-Pad1): track 0.00 -> 5.12 mm
- net /KEY_FUNC1: track 68.7 -> 72.9 mm
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- added copper zone on B.Cu, net GND
- removed copper zone on B.Cu, net VCC_MCU
Other:
- board text added: "DOWN"
- board text added: "ENTER"
- board text added: "FUNC1"
- board text added: "FUNC2"
- board text added: "JTAG"
- board text added: "LEFT"
- board text added: "MENU/ESCAPE"
- board text added: "POWER/SELECT"
- board text added: "RIGHT"
- board text added: "UP"

Commit message: pcb complete 1st
Connections:
- J1 pad 23: Net-(J1-Pad23) -> (no net)
- J1 pad 24: Net-(J1-Pad24) -> (no net)
- J1 pad 3: Net-(J1-Pad3) -> (no net)
- J1 pad 37: Net-(J1-Pad37) -> (no net)
- J1 pad 38: Net-(J1-Pad38) -> (no net)
- J1 pad 4: Net-(J1-Pad4) -> (no net)
- J2 pad 11: Net-(J2-Pad11) -> (no net)
- J2 pad 17: Net-(J2-Pad17) -> (no net)
- J2 pad 19: Net-(J2-Pad19) -> (no net)
- R5 pad 2: /KEY_POWER -> (no net)

Commit message: ...
Parts:
- R19, R20, R27: moved to F.Cu
- moved R19 5.88 mm to (167.1, 89.5), turned to 90 degrees
- moved R20 0.96 mm to (161.9, 89.5), turned to 270 degrees
Routing:
- net VCC_MCU: track 279.1 -> 2.54 mm, vias 10 -> 0
- net /TDO: track 37.0 -> 45.8 mm, vias 0 -> 2
- net /nRESET: track 37.0 -> 45.2 mm, vias 0 -> 2
- net /TMS: track 36.0 -> 42.6 mm, vias 0 -> 2
- net /TCLK: track 38.4 -> 44.0 mm, vias 1 -> 2
- net GND: track 17.8 -> 20.5 mm, vias 2 -> 9
- net /TRST: track 40.9 -> 43.0 mm, vias 1 -> 2
- net /KEY_DOWN: track 43.4 -> 41.5 mm
- net /KEY_RIGHT: track 29.7 -> 28.4 mm
- net /TDI: track 45.8 -> 45.7 mm, vias 1 -> 2
- added copper zone on F.Cu, net VCC_MCU
- removed copper zone on F.Cu, net GND

Commit message: ...
Parts:
- added G***: LOGO, FlightComputer_Library:LOGO-EAGLE-02, F.Cu at (179.4, 93.2)
- moved SW6 111.7 mm to (201.9, 83.8), turned to 180 degrees
- moved R13 110.8 mm to (92.9, 82.2), turned to 180 degrees
- moved R17 110.2 mm to (92.9, 83.8), turned to 0 degrees
- moved SW7 109.9 mm to (201.9, 96.2), turned to 180 degrees
- moved C8 109.6 mm to (92.9, 85.3), turned to 180 degrees
- moved C9 108.5 mm to (92.9, 97.8), turned to 180 degrees
- moved R18 108.3 mm to (92.9, 96.2), turned to 0 degrees
- moved R14 108.2 mm to (92.9, 94.7), turned to 180 degrees
- moved R11 101.8 mm to (196.5, 82.2), turned to 180 degrees
- moved R15 101.1 mm to (196.5, 83.8), turned to 0 degrees
- moved C6 100.5 mm to (196.5, 85.3), turned to 180 degrees
- moved SW8 99.4 mm to (98.4, 83.8), turned to 180 degrees
- moved C7 99.3 mm to (196.5, 97.8), turned to 180 degrees
- moved R16 99.1 mm to (196.5, 96.2), turned to 0 degrees
- moved R12 99.0 mm to (196.5, 94.7), turned to 180 degrees
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Connections:
- J1 pad 23: (no net) -> Net-(J1-Pad23)
- J1 pad 24: (no net) -> Net-(J1-Pad24)
- J1 pad 3: (no net) -> Net-(J1-Pad3)
- J1 pad 37: (no net) -> Net-(J1-Pad37)
- J1 pad 38: (no net) -> Net-(J1-Pad38)
- J1 pad 4: (no net) -> Net-(J1-Pad4)
- J2 pad 11: (no net) -> Net-(J2-Pad11)
- J2 pad 17: (no net) -> Net-(J2-Pad17)
- J2 pad 19: (no net) -> Net-(J2-Pad19)
- R11 pad 2: /KEY_ENTER -> /KEY_MENU
- R5 pad 2: (no net) -> /KEY_ENTER
Routing:
- net /KEY_MENU: track 2.54 -> 52.7 mm, vias 0 -> 2
- net /KEY_ENTER: track 50.4 -> 34.3 mm, vias 2 -> 0
- net /TDI: track 45.7 -> 41.9 mm
- net /KEY_DOWN: track 41.5 -> 44.9 mm
- net VCC_MCU: track 2.54 -> 0.00 mm
- net /TRST: track 43.0 -> 40.6 mm
- net /TDO: track 45.8 -> 44.7 mm
- net /KEY_RIGHT: track 28.4 -> 29.3 mm
- net /TMS: track 42.6 -> 41.8 mm
Other:
- outline, holes or cut-outs redrawn
- board text added: "ESCAPE"
- board text added: "MENU"
- board text removed: "MENU/ESCAPE"
- board text removed: "POWER/SELECT"

Commit message: ...
Routing:
- net /KEY_FUNC1: track 72.5 -> 74.6 mm

Commit message: gerber
Parts:
- removed the G*** at (179.4, 93.2)
- added G***: LOGO, FlightComputer_Library:LOGO-FC, F.Cu at (176.7, 99.7)
Routing:
- net /TCLK: track 43.8 -> 43.2 mm
