File: hw/rev1/FlightComputer-Keypad/FlightComputer-Keypad.kicad_pcb (KiCad board)
At the start: 2 copper layers, 148 x 42 mm, 48 parts, among them J1 Conn_02x20_Odd_Even, J2 Conn_02x10_Odd_Even, SW1 SW_Push, SW2 SW_Push, SW3 SW_Push, SW4 SW_Push, SW5 SW_Push, SW6 SW_Push, SW7 SW_Push, SW8 SW_Push, SW9 SW_Push

Commit message: gerber final
Parts:
- C1, C2, C3, C4, C5, C6, C7, C8, C9: footprint Capacitor_SMD:C_0402_1005Metric -> FlightComputer_Library:C_0402_1005Metric_Pad0.74x0.62mm_HandSolder
- R1, R10, R11, R12, R13, R14, R15, R16, R17, R18, R19, R2, R20, R21, R22, R23, R24, R25, R26, R27, R3, R4, R5, R6, R7, R8, R9: footprint Resistor_SMD:R_0402_1005Metric -> FlightComputer_Library:R_0402_1005Metric_Pad0.72x0.64mm_HandSolder
Routing:
- net GND: track 20.4 -> 22.2 mm, vias 9 -> 18
