File: hw/rev1/CurrentMeasure/CurrentMeasure.kicad_pcb (KiCad board)
At the start: 2 copper layers, 60 x 50 mm, 17 parts, among them J1 Conn_01x02, J2 Conn_01x02, J3 Conn_01x04, J4 Conn_01x02, J5 Conn_01x02, J6 Conn_01x02, U1 INA219AxD

Commit message: update current sensor
Parts:
- added C2: 10Uf, Capacitor_SMD:C_0603_1608Metric_Pad1.05x0.95mm_HandSolder, F.Cu at (570.0, 65.5)
- added G***: LOGO, FlightComputer:BMP-VIR, F.Cu at (547.3, 86.4)
- added G***: LOGO, FlightComputer:BMP-VIR, F.Cu at (574.3, 81.9)
- added G***: LOGO, FlightComputer:LOGO-GLIDER, F.Cu at (575.7, 79.2)
- added G***: LOGO, FlightComputer:BMP-Power-Source, F.Cu at (576.8, 54.3)
- added G***: LOGO, FlightComputer:BMP-Power-Source, F.Cu at (547.0, 55.1)
- added R10: N/C, FlightComputer:R_4527, F.Cu at (561.2, 57.1)
- J1, J6: footprint Connector_JST:JST_EH_S2B-EH_1x02_P2.50mm_Horizontal -> Connector_Molex:Molex_CLIK-Mate_502386-0270_1x02-1MP_P1.25mm_Horizontal
- R5: value 10m -> 2mR; footprint Resistor_SMD:R_2816_7142Metric_Pad3.20x4.45mm_HandSolder -> Resistor_SMD:R_2512_6332Metric_Pad1.52x3.35mm_HandSolder
- moved J2 8.78 mm to (545.0, 47.1)
- moved J1 8.70 mm to (552.0, 43.2), turned to 180 degrees
- moved J5 6.51 mm to (580.0, 47.1)
- moved J6 5.24 mm to (570.5, 43.2), turned to 180 degrees
- moved C1 1.13 mm to (570.0, 67.4)
- moved R1 1.13 mm to (570.0, 69.6)
- moved R2 1.13 mm to (570.0, 71.6)
- moved R5 0.40 mm to (561.2, 57.1)
- moved J4 0.20 mm to (563.0, 49.8)
Routing:
- net GND: track 0.00 -> 28.8 mm
- net /VOUT: track 11.0 -> 14.1 mm
- net /VIN: track 8.81 -> 11.9 mm
- net Net-(R2-Pad2): track 13.9 -> 15.2 mm
- net VCC: track 65.9 -> 66.9 mm
Other:
- board size 60 x 50 mm -> 44 x 50 mm
- board text added: "+"
- board text added: "ADDRESS: 0b10000xx"
- board text added: "H ADDR0 L"
- board text added: "H ADDR1 L"
- board text added: "INA219 Current sensor"
- board text added: "SCL"
- board text added: "SDA"
- board text added: "SHUNT"
- board text added: "Vi"
- board text added: "Vo"

Commit message: PIMIC rework finished
Parts:
- removed the G*** at (547.3, 86.4)
- removed the G*** at (574.3, 81.9)
- removed the G*** at (575.7, 79.2)
- removed the G*** at (576.8, 54.3)
- removed the G*** at (547.0, 55.1)
- added C3: 0.1uF, Capacitor_SMD:C_0603_1608Metric_Pad1.05x0.95mm_HandSolder, F.Cu at (561.2, 52.5)
- added G***: LOGO, FlighComputer:symbol-VIR, F.Cu at (575.2, 83.2)
- added G***: LOGO, FlighComputer:symbol-arrow-1, F.Cu at (576.9, 55.1)
- added G***: LOGO, FlighComputer:symbol-arrow-1, F.Cu at (547.7, 56.0)
- added J7: Conn_01x04, Connector_Molex:Molex_CLIK-Mate_502386-0470_1x04-1MP_P1.25mm_Horizontal, F.Cu at (544.9, 86.7)
Connections:
- R3 pad 1: Net-(J3-Pad2) -> Net-(J3-Pad3)
- R4 pad 1: Net-(J3-Pad3) -> Net-(J3-Pad2)
Routing:
- net Net-(J3-Pad2): track 4.12 -> 30.9 mm
- net Net-(J3-Pad3): track 4.12 -> 30.2 mm, vias 0 -> 1
- net VCC: track 66.9 -> 87.3 mm
