File: hw/rev1/FlightComputer-Booster/FlightComputer-Booster.kicad_pcb (KiCad board)
At the start: 2 copper layers, 23.1 x 20.7 mm, 16 parts, among them J1 Conn_01x02, J2 Conn_01x02, J3 Conn_01x01, U1 TPS61032PWR

Commit message: ...
Routing:
- net /LBI: track 6.45 -> 7.09 mm
Changed lines of the file:
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@@
     (thickness 1.6)
     (drawings 6)
-    (tracks 97)
+    (tracks 108)
     (zones 0)
     (modules 16)
@@
   )
   (setup
-    (last_trace_width 0.2)
+    (last_trace_width 0.25)
     (user_trace_width 0.2)
     (user_trace_width 0.25)
@@
   )
   (module FlightComputer_Library:R_0402_1005Metric_Pad0.72x0.64mm_HandSolder (layer F.Cu)
-    (at -32.25 -12.95 90)
+    (at -32.23 -12.95 90)
     (descr "Resistor SMD 0402 (1005 Metric), square (rectangular) end terminal, IPC_7351 nominal with elongated pad for handsoldering. (Body size source: IPC-SM-782 page 72, https://www.pcb-3d.com/wordpress/wp-content/uploads/ipc-sm-782a_amendment_1_and_2.pdf), generated with kicad-footprint-generator")
     (tags "resistor handsolder")
     (attr smd)
-    (fp_text reference R8 (at 0 -1.17 90) (layer F.SilkS)
+    (fp_text reference R8 (at -1.6 0 180) (layer F.SilkS)
       (effects (font (size 0.6 0.6) (thickness 0.04)))
     )
@@
     (fp_line (start 1.1 -0.47) (end 1.1 0.47) (layer F.CrtYd) (width 0.05))
     (fp_line (start 1.1 0.47) (end -1.1 0.47) (layer F.CrtYd) (width 0.05))
-    (fp_text user %R (at -1.6 -0.025 180) (layer F.Fab)
+    (fp_text user %R (at 0 -0.025 270) (layer F.Fab)
       (effects (font (size 0.6 0.6) (thickness 0.04)))
     )
@@
   )
   (module FlightComputer_Library:R_0402_1005Metric_Pad0.72x0.64mm_HandSolder (layer F.Cu)
-    (at -32.258 -15.818 90)
+    (at -32.238 -15.818 90)
     (descr "Resistor SMD 0402 (1005 Metric), square (rectangular) end terminal, IPC_7351 nominal with elongated pad for handsoldering. (Body size source: IPC-SM-782 page 72, https://www.pcb-3d.com/wordpress/wp-content/uploads/ipc-sm-782a_amendment_1_and_2.pdf), generated with kicad-footprint-generator")
     (tags "resistor handsolder")
     (attr smd)
-    (fp_text reference R4 (at 1.482 -0.042 180) (layer F.SilkS)
+    (fp_text reference R4 (at 1.532 0.008 180) (layer F.SilkS)
       (effects (font (size 0.6 0.6) (thickness 0.04)))
     )
@@
     (fp_line (start 1.08 -0.46) (end 1.08 0.46) (layer F.CrtYd) (width 0.05))
     (fp_line (start 1.08 0.46) (end -1.08 0.46) (layer F.CrtYd) (width 0.05))
-    (fp_text user %R (at -1.75 -0.021) (layer F.Fab)
+    (fp_text user %R (at 0 0.004) (layer F.Fab)
       (effects (font (size 0.6 0.6) (thickness 0.04)))
     )
@@
   (segment (start -30.6 -16.32) (end -30.86 -16.06) (width 0.25) (layer F.Cu) (net 3))
   (segment (start -30.86 -16.06) (end -30.86 -15.35) (width 0.25) (layer F.Cu) (net 3))
-  (segment (start -30.9895 -15.2205) (end -32.258 -15.2205) (width 0.25) (layer F.Cu) (net 3))
   (segment (start -30.86 -15.35) (end -30.9895 -15.2205) (width 0.25) (layer F.Cu) (net 3))
   (segment (start -29.2325 -19.3925) (end -29 -19.625) (width 0.5) (layer F.Cu) (net 3))
   (segment (start -29.2325 -18.796) (end -29.2325 -19.3925) (width 0.5) (layer F.Cu) (net 3))
   (segment (start -29 -20.3) (end -29 -19.625) (width 0.5) (layer F.Cu) (net 3))
+  (segment (start -32.238 -15.2205) (end -30.9895 -15.2205) (width 0.25) (layer F.Cu) (net 3))
   (segment (start -32.766 -10.16) (end -33.525 -10.919) (width 0.25) (layer F.Cu) (net 4))
   (segment (start -32.766 -8.382) (end -32.766 -10.16) (width 0.25) (layer F.Cu) (net 4))
   (segment (start -33.525 -12.3525) (end -33.525 -10.919) (width 0.25) (layer F.Cu) (net 4))
-  (segment (start -30.535 -11.703) (end -32.053 -11.703) (width 0.25) (layer F.Cu) (net 5))
-  (segment (start -32.25 -11.9) (end -32.25 -12.3525) (width 0.25) (layer F.Cu) (net 5))
-  (segment (start -32.053 -11.703) (end -32.25 -11.9) (width 0.25) (layer F.Cu) (net 5))
-  (segment (start -33.445 -13.5475) (end -32.25 -12.3525) (width 0.25) (layer F.Cu) (net 5))
-  (segment (start -33.525 -13.5475) (end -33.445 -13.5475) (width 0.25) (layer F.Cu) (net 5))
+  (segment (start -32.053 -11.703) (end -30.535 -11.703) (width 0.25) (layer F.Cu) (net 5))
+  (segment (start -32.25 -11.9) (end -32.053 -11.703) (width 0.25) (layer F.Cu) (net 5))
+  (segment (start -32.25 -12.3525) (end -32.25 -11.9) (width 0.25) (layer F.Cu) (net 5))
+  (segment (start -32.87501 -13.36501) (end -32.87501 -12.59499) (width 0.25) (layer F.Cu) (net 5))
+  (segment (start -33.0575 -13.5475) (end -32.87501 -13.36501) (width 0.25) (layer F.Cu) (net 5))
+  (segment (start -33.525 -13.5475) (end -33.0575 -13.5475) (width 0.25) (layer F.Cu) (net 5))
+  (segment (start -32.63252 -12.3525) (end -32.87501 -12.59499) (width 0.25) (layer F.Cu) (net 5))
+  (segment (start -32.23 -12.3525) (end -32.63252 -12.3525) (width 0.25) (layer F.Cu) (net 5))
   (segment (start -27.94 -7.8825) (end -28.2925 -7.8825) (width 0.25) (layer F.Cu) (net 6))
   (segment (start -28.2925 -7.8825) (end -28.56499 -8.15499) (width 0.25) (layer F.Cu) (net 6))
@@
   (segment (start -28.585 -10.315) (end -28.585 -11.703) (width 0.25) (layer F.Cu) (net 6))
   (segment (start -29.21 -9.69) (end -28.585 -10.315) (width 0.25) (layer F.Cu) (net 6))
-  (segment (start -33.453 -15.2205) (end -32.258 -16.4155) (width 0.25) (layer F.Cu) (net 7))
   (segment (start -33.528 -15.2205) (end -33.453 -15.2205) (width 0.25) (layer F.Cu) (net 7))
-  (segment (start -32.258 -17.872) (end -32.258 -16.4155) (width 0.25) (layer F.Cu) (net 7))
-  (segment (start -31.96901 -18.16099) (end -32.258 -17.872) (width 0.25) (layer F.Cu) (net 7))
   (segment (start -30.18099 -18.16099) (end -31.96901 -18.16099) (width 0.25) (layer F.Cu) (net 7))
   (segment (start -29.885 -17.865) (end -30.18099 -18.16099) (width 0.25) (layer F.Cu) (net 7))
   (segment (start -29.885 -17.253) (end -29.885 -17.865) (width 0.25) (layer F.Cu) (net 7))
+  (segment (start -32.238 -17.892) (end -31.96901 -18.16099) (width 0.25) (layer F.Cu) (net 7))
+  (segment (start -32.238 -16.4155) (end -32.238 -17.892) (width 0.25) (layer F.Cu) (net 7))
+  (segment (start -32.238 -16.4155) (end -32.75749 -16.4155) (width 0.25) (layer F.Cu) (net 7))
+  (segment (start -32.88 -15.62191) (end -32.88301 -15.6189) (width 0.25) (layer F.Cu) (net 7))
+  (segment (start -32.88301 -15.6189) (end -32.88301 -15.35699) (width 0.25) (layer F.Cu) (net 7))
+  (segment (start -33.0195 -15.2205) (end -33.528 -15.2205) (width 0.25) (layer F.Cu) (net 7))
+  (segment (start -32.88301 -15.35699) (end -33.0195 -15.2205) (width 0.25) (layer F.Cu) (net 7))
+  (segment (start -32.88301 -16.01708) (end -32.88299 -16.0171) (width 0.25) (layer F.Cu) (net 7))
+  (segment (start -32.88301 -15.6189) (end -32.88301 -16.01708) (width 0.25) (layer F.Cu) (net 7))
+  (segment (start -32.88299 -16.29) (end -32.75749 -16.4155) (width 0.25) (layer F.Cu) (net 7))
+  (segment (start -32.88299 -16.0171) (end -32.88299 -16.29) (width 0.25) (layer F.Cu) (net 7))
   (segment (start -26.635 -17.253) (end -25.985 -17.253) (width 0.4) (layer F.Cu) (net 8))
   (zone (net 1) (net_name GND) (layer F.Cu) (hatch edge 0.508)
@@
   (zone (net 3) (net_name VCC_BAT) (layer F.Cu) (hatch edge 0.508)
     (priority 2)
-    (connect_pads (clearance 0.2))
+    (connect_pads yes (clearance 0.2))
     (min_thickness 0.2)
     (fill yes (arc_segments 32) (thermal_gap 0.2) (thermal_bridge_width 0.6))
     (polygon
       (pts
-        (xy -6.1 -16.475) (xy -29.75 -16.45) (xy -29.75 -29.325) (xy -6.1 -29.325)
+        (xy -6.1 -16.9) (xy -29.6 -16.9) (xy -29.6 -29.3) (xy -6.1 -29.325)
       )
     )
@@
     (polygon
       (pts
-        (xy -3.6 -11.9) (xy -25.2 -11.9) (xy -25.2 -15.875) (xy -27 -15.9) (xy -27 -18.8)
-        (xy -3.6 -18.8)
+        (xy -3.6 -11.9) (xy -23.2 -11.9) (xy -23.2 -13.7) (xy -27 -13.7) (xy -27 -18.4)
+        (xy -3.6 -18.4)
       )
     )
@@
   (zone (net 2) (net_name VCC_5V) (layer F.Cu) (hatch edge 0.508)
     (priority 3)
-    (connect_pads (clearance 0.2))
+    (connect_pads yes (clearance 0.2))
     (min_thickness 0.2)
-    (fill yes (arc_segments 32) (thermal_gap 0.24) (thermal_bridge_width 0.6))
+    (fill yes (arc_segments 32) (thermal_gap 0.24) (thermal_bridge_width 0.5))
     (polygon
       (pts
-        (xy -25.7 -12.4) (xy -25.7 -11.7) (xy -6.8 -11.7) (xy -6.8 -3) (xy -14.5 -3)
-        (xy -14.5 -8.4) (xy -18 -8.4) (xy -18 -7.3) (xy -25.75 -7.3) (xy -25.75 -8.5)
-        (xy -28.7 -8.5) (xy -28.7 -10.7) (xy -28.7 -12.4)
+        (xy -25.7 -11.9) (xy -25.7 -11.7) (xy -6.8 -11.7) (xy -6.8 -3) (xy -14 -3)
+        (xy -14 -8.1) (xy -17.7 -8.1) (xy -17.7 -7.3) (xy -25.5 -7.3) (xy -25.5 -9)
+        (xy -28.1 -9) (xy -28.1 -11.6) (xy -28.1 -11.9)
       )
     )
