File: hw/rev1/EINKPower/EINKPower.kicad_pcb (KiCad board)
At the start: 2 copper layers, 30 x 20 mm, 40 parts, among them J1 Conn_01x02, J2 Conn_01x02, J3 Conn_01x02, J4 Conn_01x02, J5 Conn_01x03, U1 LT1945, U2 LM358, U3 MC78L15_SO8, U4 MC79L15_SO8

Commit message: ...
Parts:
- removed the C1 at (-521.5, -272.5)
- removed C12, C13: 10uF, Capacitor_Tantalum_SMD:CP_EIA-1608-08_AVX-J_Pad1.25x1.05mm_HandSolder
- removed the C7 at (-532.5, -265.0)
- removed the C8 at (-514.0, -285.2)
- removed the U2 at (-521.2, -277.0)
- added C2: 4.7uF, Capacitor_SMD:C_0805_2012Metric_Pad1.15x1.40mm_HandSolder, F.Cu at (144.8, 86.8)
- added J6: Conn_01x01, Connector_PinHeader_1.27mm:PinHeader_1x01_P1.27mm_Vertical, F.Cu at (156.7, 93.3)
- added J7: Conn_01x01, Connector_PinHeader_1.27mm:PinHeader_1x01_P1.27mm_Vertical, F.Cu at (160.8, 90.0)
- added J8: Conn_01x01, Connector_PinHeader_1.27mm:PinHeader_1x01_P1.27mm_Vertical, F.Cu at (160.8, 93.3)
- added J9: Conn_01x01, Connector_PinHeader_1.27mm:PinHeader_1x01_P1.27mm_Vertical, F.Cu at (164.9, 90.0)
- added U1: LM358, Package_SO:TSSOP-8_3x3mm_P0.65mm, F.Cu at (118.9, 100.0)
- C1: renamed from C15; footprint FlightComputer_Library:C_0402_1005Metric_Pad0.74x0.62mm_HandSolder -> Capacitor_SMD:C_0603_1608Metric_Pad1.05x0.95mm_HandSolder
- C10: renamed from C9; value 0.1uF -> 4.7uF; footprint FlightComputer_Library:C_0402_1005Metric_Pad0.74x0.62mm_HandSolder -> Capacitor_SMD:C_0603_1608Metric_Pad1.05x0.95mm_HandSolder
- C11: value 0.1uF -> 1uF; footprint FlightComputer_Library:C_0402_1005Metric_Pad0.74x0.62mm_HandSolder -> Capacitor_SMD:C_0603_1608Metric_Pad1.05x0.95mm_HandSolder
- C14: renamed from C10; value 0.1uF -> 4.7uF; footprint FlightComputer_Library:C_0402_1005Metric_Pad0.74x0.62mm_HandSolder -> Capacitor_SMD:C_0603_1608Metric_Pad1.05x0.95mm_HandSolder
- C16: renamed from C14; value 0.1uF -> 1uF; footprint FlightComputer_Library:C_0402_1005Metric_Pad0.74x0.62mm_HandSolder -> Capacitor_SMD:C_0603_1608Metric_Pad1.05x0.95mm_HandSolder
- C3, C6: footprint FlightComputer_Library:C_0402_1005Metric_Pad0.74x0.62mm_HandSolder -> Capacitor_SMD:C_0603_1608Metric_Pad1.05x0.95mm_HandSolder
- C4: renamed from C5; footprint FlightComputer_Library:C_0402_1005Metric_Pad0.74x0.62mm_HandSolder -> Capacitor_SMD:C_0603_1608Metric_Pad1.05x0.95mm_HandSolder
- C5: renamed from C16; footprint FlightComputer_Library:C_0402_1005Metric_Pad0.74x0.62mm_HandSolder -> Capacitor_SMD:C_0603_1608Metric_Pad1.05x0.95mm_HandSolder
- C7: renamed from C4; footprint FlightComputer_Library:C_0402_1005Metric_Pad0.74x0.62mm_HandSolder -> Capacitor_SMD:C_0603_1608Metric_Pad1.05x0.95mm_HandSolder
- C8: renamed from C2; footprint FlightComputer_Library:C_0402_1005Metric_Pad0.74x0.62mm_HandSolder -> Capacitor_SMD:C_0603_1608Metric_Pad1.05x0.95mm_HandSolder
- J1, J2, J3, J4: value Conn_01x02 -> Conn_01x01; footprint Connector_PinHeader_2.54mm:PinHeader_1x02_P2.54mm_Vertical -> Connector_PinHeader_1.27mm:PinHeader_1x01_P1.27mm_Vertical
- J5: value Conn_01x03 -> Conn_01x01; footprint Connector_PinHeader_2.54mm:PinHeader_1x03_P2.54mm_Vertical -> Connector_PinHeader_1.27mm:PinHeader_1x01_P1.27mm_Vertical
- L1, L2: footprint Inductor_SMD:L_12x12mm_H6mm -> Inductor_SMD:L_6.3x6.3_H3
- R1: renamed from R5; footprint FlightComputer_Library:R_0402_1005Metric_Pad0.72x0.64mm_HandSolder -> Resistor_SMD:R_0603_1608Metric_Pad0.98x0.95mm_HandSolder
- R2: renamed from R9; footprint FlightComputer_Library:R_0402_1005Metric_Pad0.72x0.64mm_HandSolder -> Resistor_SMD:R_0603_1608Metric_Pad0.98x0.95mm_HandSolder
- R3: renamed from R6; footprint FlightComputer_Library:R_0402_1005Metric_Pad0.72x0.64mm_HandSolder -> Resistor_SMD:R_0603_1608Metric_Pad0.98x0.95mm_HandSolder
- R4: renamed from R1; footprint FlightComputer_Library:R_0402_1005Metric_Pad0.72x0.64mm_HandSolder -> Resistor_SMD:R_0603_1608Metric_Pad0.98x0.95mm_HandSolder
- R5: renamed from R2; footprint FlightComputer_Library:R_0402_1005Metric_Pad0.72x0.64mm_HandSolder -> Resistor_SMD:R_0603_1608Metric_Pad0.98x0.95mm_HandSolder
- R6: renamed from R3; footprint FlightComputer_Library:R_0402_1005Metric_Pad0.72x0.64mm_HandSolder -> Resistor_SMD:R_0603_1608Metric_Pad0.98x0.95mm_HandSolder
- R7: renamed from R4; footprint FlightComputer_Library:R_0402_1005Metric_Pad0.72x0.64mm_HandSolder -> Resistor_SMD:R_0603_1608Metric_Pad0.98x0.95mm_HandSolder
- R8: renamed from R7; footprint FlightComputer_Library:R_0402_1005Metric_Pad0.72x0.64mm_HandSolder -> Resistor_SMD:R_0603_1608Metric_Pad0.98x0.95mm_HandSolder
- R9: renamed from R8; footprint FlightComputer_Library:R_0402_1005Metric_Pad0.72x0.64mm_HandSolder -> Resistor_SMD:R_0603_1608Metric_Pad0.98x0.95mm_HandSolder
- RV1: footprint Potentiometer_THT:Potentiometer_Bourns_3299W_Vertical -> Potentiometer_SMD:Potentiometer_Bourns_3214J_Horizontal
- moved L2 786.6 mm to (139.5, 103.8), turned to 270 degrees
- moved L1 786.2 mm to (139.0, 89.5), turned to 270 degrees
- moved J5 779.1 mm to (146.0, 100.2), turned to 90 degrees
- moved J4 778.7 mm to (156.7, 90.0)
- moved D1 774.7 mm to (133.8, 95.8)
- moved D3 773.8 mm to (133.2, 86.4)
- moved D2 772.6 mm to (133.2, 88.0), turned to 180 degrees
- moved J2 770.8 mm to (152.5, 93.3)
- moved R6 769.2 mm to (149.5, 98.2)
- moved J3 768.7 mm to (146.0, 93.8), turned to 90 degrees
- moved J1 768.3 mm to (152.5, 90.0)
- moved R4 768.3 mm to (145.2, 98.0)
- moved U2 767.0 mm to (139.8, 97.0), turned to 180 degrees
- moved R1 765.6 mm to (129.6, 101.1)
- moved R8 765.4 mm to (128.8, 108.1)
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- renumbered U1 to U2
Connections:
- J1 pad 1: VCC_5V -> +22V
- J2 pad 1: -20V -> VCC_5V
- J3 pad 1: -15V -> /EN_VDD
- J4 pad 1: GND -> -20V
- J5 pad 1: /EN_VDD -> /EN_VEE
Routing:
- removed copper zone on B.Cu, net GND
Other:
- board size 30 x 20 mm -> 35 x 27.8 mm
