File: hw/rev1/CurrentSensor/CurrentMeasure.kicad_pcb (KiCad board)
At the start: 2 copper layers, 44 x 50 mm, 24 parts, among them J1 Conn_01x02, J2 Conn_01x02, J3 Conn_01x04, J4 Conn_01x02, J5 Conn_01x02, J6 Conn_01x02, J7 Conn_01x04, U1 INA219AxD

Commit message: fixed miss connection
Connections:
- J7 pad 4: Net-(J7-Pad4) -> GND
